File: powerSwitch/pcb/CNC-PowerSwitch-2016-v0.9.brd (EAGLE design)
At the start: 53.3 x 99.7 mm, 111 parts, among them IC10 BTS6133, IC11 BTS6133, IC12 BTS6133, IC15 BTS6133, IC4 BTS555, P1 39-30-06?_S, P4 39-30-06?_S, P6 39-30-04?_S, P8 39-30-04?_S, Q1 16Mhz, T1 BC847, T2 BC849, T3 BC849, T4 BC859, T5 BC849, T6 BC849, T7 BC849, U1 LM2675M

Commit message: PowerSwitch PartList
Parts:
- C1, C14, C16, C24, C5: value 100n -> 100n/10V
- C10, C11: value 22p -> 22p/10V
- L2: value 100µ -> 68µ
- OK1: value ACPL-227-500E -> ILD213T
- R35: value 220k 0.1% -> 240k 0.1%
- R4: value 150 -> 120
- T1: value BC847 -> BC849
Other:
- board text added: "info@das-lab.net"
Changed lines of the file:
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@@
 </polygon>
 <text x="31.115" y="96.139" size="1.016" layer="25">2016 v0.9</text>
+<text x="31.115" y="94.615" size="1.016" layer="25">info@das-lab.net</text>
 </plain>
 <attributes>
@@
 <attribute name="MF" value="" x="8.509" y="86.741" size="1.778" layer="27" rot="R180" display="off"/>
 </element>
-<element name="C10" library="rcl" package="C0603" value="22p" x="6.223" y="82.931" rot="R180"/>
-<element name="C11" library="rcl" package="C0603" value="22p" x="10.795" y="82.931"/>
-<element name="C14" library="rcl" package="C0603" value="100n" x="13.081" y="69.596" smashed="yes" rot="MR270">
+<element name="C10" library="rcl" package="C0603" value="22p/10V" x="6.223" y="82.931" rot="R180"/>
+<element name="C11" library="rcl" package="C0603" value="22p/10V" x="10.795" y="82.931"/>
+<element name="C14" library="rcl" package="C0603" value="100n/10V" x="13.081" y="69.596" smashed="yes" rot="MR270">
 <attribute name="NAME" x="12.431" y="70.396" size="1.016" layer="26" rot="MR270"/>
 <attribute name="VALUE" x="14.731" y="70.396" size="1.016" layer="28" rot="MR270"/>
@@
 <attribute name="OC_NEWARK" value="unknown" x="5.08" y="31.496" size="1.778" layer="27" rot="R90" display="off"/>
 </element>
-<element name="T1" library="transistor" package="SOT23" value="BC847" x="9.906" y="53.467" smashed="yes" rot="MR0">
-<attribute name="NAME" x="11.811" y="55.372" size="1.27" layer="26" rot="MR0"/>
-<attribute name="VALUE" x="11.811" y="50.292" size="1.27" layer="28" rot="MR0"/>
-</element>
 <element name="R5" library="rcl" package="R0805" value="4k7" x="10.287" y="60.96" smashed="yes" rot="MR270">
 <attribute name="NAME" x="11.049" y="57.785" size="1.27" layer="26" rot="MR270"/>
 <attribute name="VALUE" x="12.827" y="61.595" size="1.27" layer="28" rot="MR270"/>
 </element>
-<element name="C16" library="rcl" package="C0603" value="100n" x="9.525" y="69.596" smashed="yes" rot="MR90">
+<element name="C16" library="rcl" package="C0603" value="100n/10V" x="9.525" y="69.596" smashed="yes" rot="MR90">
 <attribute name="NAME" x="10.175" y="68.796" size="1.016" layer="26" rot="MR90"/>
 <attribute name="VALUE" x="7.875" y="68.796" size="1.016" layer="28" rot="MR90"/>
 </element>
-<element name="C24" library="rcl" package="C0603" value="100n" x="2.159" y="17.018" smashed="yes" rot="MR270">
+<element name="C24" library="rcl" package="C0603" value="100n/10V" x="2.159" y="17.018" smashed="yes" rot="MR270">
 <attribute name="NAME" x="2.921" y="15.494" size="1.27" layer="26" rot="MR90"/>
 <attribute name="VALUE" x="4.191" y="17.907" size="1.27" layer="28" rot="MR270"/>
@@
 <element name="H7" library="holes" package="3,0-PAD" value="MOUNT-PAD-ROUND3.0" x="3.984" y="3.984" locked="yes"/>
 <element name="H8" library="holes" package="3,0-PAD" value="MOUNT-PAD-ROUND3.0" x="49.332" y="3.984" locked="yes"/>
-<element name="C5" library="rcl" package="C0603" value="100n" x="11.303" y="69.596" rot="MR90"/>
+<element name="C5" library="rcl" package="C0603" value="100n/10V" x="11.303" y="69.596" rot="MR90"/>
 <element name="R15" library="rcl" package="R0805" value="100k" x="39.497" y="13.843" rot="MR270"/>
 <element name="R16" library="rcl" package="R0805" value="100k" x="32.639" y="13.843" rot="MR270"/>
@@
 <element name="VR6" library="1_USER" package="SOT23" value="TL431_SOT23" x="20.193" y="34.671" rot="MR0"/>
 <element name="R30" library="rcl" package="R0805" value="100k 0.1%" x="21.209" y="29.591" rot="MR90"/>
-<element name="R35" library="rcl" package="R0805" value="220k 0.1%" x="23.495" y="29.591" rot="MR270"/>
+<element name="R35" library="rcl" package="R0805" value="240k 0.1%" x="23.495" y="29.591" rot="MR270"/>
 <element name="VR7" library="1_USER" package="SOT23" value="TL431_SOT23" x="36.576" y="50.292" rot="MR270"/>
 <element name="R36" library="rcl" package="R0805" value="100k 0.1%" x="43.434" y="51.054" rot="MR0"/>
@@
 <attribute name="OC_FARNELL" value="unknown" x="14.605" y="31.496" size="1.778" layer="27" rot="R90" display="off"/>
 </element>
-<element name="C1" library="rcl" package="C0603" value="100n" x="7.239" y="53.467" rot="MR270"/>
+<element name="C1" library="rcl" package="C0603" value="100n/10V" x="7.239" y="53.467" rot="MR270"/>
 <element name="F1" library="fuse" package="TE5" value="FUSETE5" x="37.719" y="27.178">
 <attribute name="MPN" value="" x="37.719" y="27.178" size="1.778" layer="27" display="off"/>
@@
 <element name="C2" library="rcl" package="PANASONIC_D" value="47µ/35V" x="48.006" y="12.065"/>
 <element name="C3" library="rcl" package="PANASONIC_D" value="47µ/35V" x="40.132" y="19.812" rot="R90"/>
-<element name="L2" library="Inductor-Fastron" package="PISM" value="100µ" x="45.339" y="18.923" rot="MR180"/>
+<element name="L2" library="Inductor-Fastron" package="PISM" value="68µ" x="45.339" y="18.923" rot="MR180"/>
 <element name="C4" library="rcl" package="C0603" value="10n/35V" x="50.038" y="20.32" rot="R270"/>
 <element name="D2" library="diode" package="SMA-DO214AC" value="ES1A" x="48.006" y="12.065" rot="MR180"/>
@@
 <element name="R1" library="rcl" package="R0805" value="50k" x="28.321" y="6.223" rot="MR270"/>
 <element name="T3" library="transistor" package="SOT23" value="BC849" x="33.274" y="4.064" rot="MR180"/>
-<element name="R4" library="rcl" package="R0805" value="150" x="33.274" y="9.017" rot="R270"/>
+<element name="R4" library="rcl" package="R0805" value="120" x="33.274" y="9.017" rot="R270"/>
 <element name="LED_BLAU" library="led" package="CHIPLED_0805" value="" x="33.274" y="4.064" rot="R180"/>
 <element name="R7" library="rcl" package="R0805" value="50k" x="21.971" y="6.223" rot="MR90"/>
@@
 <element name="D10" library="DB2430700L" package="TMINIP2-F2-B" value="DB2430700L" x="27.051" y="41.656" rot="R90"/>
 <element name="D11" library="DB2430700L" package="TMINIP2-F2-B" value="DB2430700L" x="30.353" y="41.656" rot="R90"/>
-<element name="OK1" library="optocoupler" package="SOIC08" value="ACPL-227-500E" x="22.479" y="37.338" rot="R180">
+<element name="OK1" library="optocoupler" package="SOIC08" value="ILD213T" x="22.479" y="37.338" rot="R180">
 <attribute name="MPN" value="ILD207T" x="22.479" y="37.338" size="1.778" layer="27" rot="R180" display="off"/>
 <attribute name="OC_FARNELL" value="1469603" x="22.479" y="37.338" size="1.778" layer="27" rot="R180" display="off"/>
@@
 <element name="P8" library="con-molex-mini-fit" package="39-30-?04?" value="39-30-04?_S" x="39.37" y="85.979" rot="R90"/>
 <element name="P1" library="con-molex-mini-fit" package="39-30-?06?" value="39-30-06?_S" x="39.37" y="37.338" rot="R90"/>
+<element name="T1" library="transistor" package="SOT23" value="BC849" x="9.906" y="53.467" rot="MR0"/>
 </elements>
 <signals>
@@
 </signal>
 <signal name="GND">
-<contactref element="T1" pad="2"/>
 <contactref element="C24" pad="1"/>
 <contactref element="R2" pad="1"/>
@@
 <via x="4.572" y="48.641" extent="1-16" drill="0.5"/>
 <via x="19.05" y="51.943" extent="1-16" drill="0.5"/>
+<contactref element="T1" pad="2"/>
 </signal>
 <signal name="N$10">
@@
 </signal>
 <signal name="N$1">
-<contactref element="T1" pad="1"/>
 <contactref element="R5" pad="2"/>
 <wire x1="10.287" y1="60.01" x2="10.287" y2="56.007" width="0.254" layer="16"/>
 <wire x1="10.287" y1="56.007" x2="10.856" y2="55.438" width="0.254" layer="16"/>
-<wire x1="10.856" y1="52.367" x2="10.856" y2="55.438" width="0.254" layer="16"/>
+<contactref element="T1" pad="1"/>
+<wire x1="10.856" y1="55.438" x2="10.856" y2="52.367" width="0.254" layer="16"/>
 </signal>
 <signal name="N$20">
+<contactref element="TDB-05" pad="-"/>
 <contactref element="T1" pad="3"/>
-<contactref element="TDB-05" pad="-"/>
-<wire x1="7.239" y1="57.277" x2="7.239" y2="57.234" width="0.254" layer="16"/>
-<wire x1="7.239" y1="57.234" x2="9.906" y2="54.567" width="0.254" layer="16"/>
+<wire x1="9.906" y1="54.567" x2="9.906" y2="54.61" width="0.4064" layer="16"/>
+<wire x1="9.906" y1="54.61" x2="7.239" y2="57.277" width="0.4064" layer="16"/>
 </signal>
 <signal name="TXCAN">
