File: powerSwitch/pcb/CNC-PowerSwitch-2016-v0.9.sch (EAGLE design)
At the start: 111 parts, among them IC10 BTS6133, IC11 BTS6133, IC12 BTS6133, IC15 BTS6133, IC4 BTS555, P1 39-30-06_S, P4 39-30-06_S, P6 39-30-04_S, P8 39-30-04_S, Q1 16Mhz, T1 BC847, T2 BC849, T3 BC849, T4 BC859, T5 BC849, T6 BC849, T7 BC849, U1 LM2675M

Commit message: PowerSwitch PartList
Parts:
- C1, C14, C16, C24, C5: value 100n -> 100n/10V
- C10, C11: value 22p -> 22p/10V
- L2: value 100µ -> 68µ
- OK1: value ACPL-227-500E -> ILD213T
- R35: value 220k 0.1% -> 240k 0.1%
- R4: value 150 -> 120
- T1: value BC847 -> BC849; device transistor:BC847 -> transistor:BC849
Other:
- moved on the sheet: C10, C11, C14, P1, P1-2, P1-3, P1-4, P1-5, P1-6, P4, P4-2, P4-3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
