File: powerSwitch/pcb/CNC-PowerSwitch-2016-v0.92.brd (EAGLE design)
At the start: 53.3 x 99.7 mm, 114 parts, among them IC1 LM1458D, IC11 BTS6133, IC12 BTS6133, IC4 BTS555, P1 39-30-06?_S, P4 39-30-06?_S, P6 39-30-04?_S, P8 39-30-04?_S, Q1 16Mhz, Q2 IRF9530, Q3 IRF9530, Q4 IRF9530, Q5 IRF9530, T1 BC849, T2 BC849, T3 BC849, T4 BC859, T5 BC849, T6 BC849, T7 BC849, U1 LM2675M

Commit message: powerswitch final version and partlist
Parts:
- R12: value 0.001 -> 0.002; device rcl:R0805 -> rcl:R2512
- moved R12 1.78 mm to (45.3, 37.3)
Routing:
- net +5V: track 226.1 -> 226.9 mm, vias 8 -> 9
- net 12V-EXT: track 82.2 -> 82.7 mm
Other:
- board text added: "CNC PowerSwitch 2016 v0.92 info@das-lab.net"
- board text removed: "2016 v0.9"
- board text removed: "CNC PowerSwitch"
- board text removed: "info@das-lab.net"
