File: powerSwitch/pcb/CNC-PowerSwitch-2016-v0.92.sch (EAGLE design)
At the start: 114 parts, among them IC1 LM1458D, IC11 BTS6133, IC12 BTS6133, IC4 BTS555, P1 39-30-06_S, P4 39-30-06_S, P6 39-30-04_S, P8 39-30-04_S, Q1 16Mhz, Q2 IRF9530, Q3 IRF9530, Q4 IRF9530, Q5 IRF9530, T1 BC849, T2 BC849, T3 BC849, T4 BC859, T5 BC849, T6 BC849, T7 BC849, U1 LM2675M

Commit message: powerswitch final version and partlist
Parts:
- R12: value 0.001 -> 0.002; device rcl:R-EU_R0805 -> rcl:R-EU_R2512
Changed lines of the file:
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@@
 <part name="Q4" library="transistor-power" deviceset="IRF9530" device=""/>
 <part name="Q5" library="transistor-power" deviceset="IRF9530" device=""/>
-<part name="R12" library="rcl" deviceset="R-EU_" device="R0805" value="0.001"/>
+<part name="R12" library="rcl" deviceset="R-EU_" device="R2512" value="0.002"/>
 <part name="IC1" library="linear" deviceset="*1458" device="D" technology="LM"/>
 <part name="VR1" library="1_USER" deviceset="TL431" device="_SOT23"/>
@@
 <wire x1="22.86" y1="20.32" x2="25.4" y2="20.32" width="0.1524" layer="91"/>
 <pinref part="P1" gate="-2" pin="P"/>
-</segment>
-</net>
+<label x="38.1" y="20.32" size="1.778" layer="95"/>
+</segment>
+</net>
