File: powerSwitch/pcb/CNC-PowerSwitch-2016-v0.95.brd (EAGLE design)
At the start: 70 x 99.7 mm, 102 parts, among them IC1 LM1458D, IC11 BTS6133, IC12 BTS6133, IC2 R-78E3.3-0.5, IC3 R-78E5.0-0.5, IC4 BTS555, P1 39-30-06?_S, P4 39-30-06?_S, P6 39-30-04?_S, P8 39-30-04?_S, Q1 16Mhz, Q2 IRF9530, Q3 IRF9530, Q4 IRF9530, Q5 IRF9530, T1 BC849, U2 TXB0108PWR

Commit message: powerswitch added ethernet, next step design
Parts:
- removed D3: ES1A, diode:SMA-DO214AC
- removed OK1: ILD213, optocoupler:SOIC08
- removed R32: 1k, rcl:R0805
- added C9: 1000µ/35V, rcl:E5-10,5
- added D2: ES1A, diode:SMA-DO214AC
- added KK1, KK2: SK104, heatsink:SK104
- added Q6, Q7: BSS84, transistor-pnp:SOT23-BEC
- added R26, R7: 10k, rcl:R0805
- added U$3, U$4, U$5, U$6: SK95-2M3, modifiedHeatsinks:SK95-2M3
- T1: value BC849 -> NX7002BK
- moved VR3 57.9 mm to (100.6, 11.2)
- moved R42 56.5 mm to (97.9, 11.4)
- moved R30 55.7 mm to (92.1, 9.78)
- moved R34 55.7 mm to (94.9, 33.3)
- moved R35 55.7 mm to (94.4, 9.78)
- moved R45 55.7 mm to (89.9, 24.0)
- moved R46 55.7 mm to (89.9, 18.7)
- moved VR1 55.7 mm to (89.9, 28.7)
- moved VR2 55.7 mm to (91.9, 9.53)
- moved D1 52.0 mm to (77.9, 17.9), flipped to the top, turned to 0 degrees
- moved R13 11.1 mm to (23.7, 61.7), turned to 0 degrees
- moved R21 11.1 mm to (23.7, 61.7), turned to 0 degrees
- moved Q4 10.9 mm to (50.5, 24.6), turned to 180 degrees
- moved Q5 8.82 mm to (38.1, 29.7), turned to 270 degrees
- moved R2 8.29 mm to (23.7, 57.1), turned to 180 degrees
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Connections:
- removed net N$18: OK1.7, VR1.1
- removed net N$19: OK1.2, OK1.3
- removed net N$32: OK1.5, VR3.1
- removed net N$35: D1.K, D3.K, R32.2
- new net N$2: Q7.C, VR1.1
- new net N$8: Q6.C, VR3.1
- new net N$9: D2.A, R7.2
- net 12V: now also C9.+
- net 12V-AKKU: now also R7.1; no longer D3.A
- net 12V-EXT: now also R26.1; no longer D1.A
- net GND: now also C9.-, U2.11
- net N$12: now also D1.A, R26.2; no longer OK1.1, R32.1
- net N$30: now also Q6.E; no longer OK1.6
- net N$49: now also Q7.E; no longer OK1.8
- net SW_12V: now also D1.K, D2.K, Q6.B, Q7.B; no longer OK1.4
Routing:
- net INT_ETH: track 0.00 -> 54.4 mm, vias 0 -> 1
- net WOL_ETH: track 0.00 -> 53.7 mm, vias 0 -> 1
- net SCK: track 0.00 -> 52.1 mm, vias 0 -> 1
- net CLKOUT_ETH: track 0.00 -> 49.8 mm, vias 0 -> 1
- net CS_ETH: track 0.00 -> 48.3 mm, vias 0 -> 1
- net RST_ETH: track 0.00 -> 45.2 mm, vias 0 -> 1
- net N$11: track 0.00 -> 22.5 mm
- net N$10: track 0.00 -> 18.7 mm
- net MISO: track 0.00 -> 18.1 mm, vias 0 -> 1
- net MOSI: track 0.00 -> 17.9 mm, vias 0 -> 1

Commit message: powerswitch layout
Parts:
- moved C24 3.53 mm to (8.64, 15.9)
- moved R31 3.53 mm to (10.8, 9.53)
- moved U$1 3.53 mm to (12.7, 15.9)
Routing:
- net +3V3: track 0.00 -> 55.9 mm
- net +5V: track 0.00 -> 51.0 mm, vias 0 -> 1
- net N$22: track 0.00 -> 32.4 mm
- net TXCAN: track 0.00 -> 25.2 mm
- net CLKOUT_ETH_3V: track 0.00 -> 25.1 mm
- net RXCAN: track 0.00 -> 23.3 mm
- net CS_ETH_3V: track 0.00 -> 22.4 mm
- net 12V: track 0.00 -> 22.0 mm
- net RST_ETH_3V: track 0.00 -> 19.7 mm
- net SCK_3V: track 0.00 -> 17.5 mm
- net MOSI_3V: track 0.00 -> 14.7 mm
- net MISO_3V: track 0.00 -> 11.9 mm
- net WOL_ETH_3V: track 0.00 -> 9.10 mm
- net INT_ETH_3V: track 0.00 -> 6.03 mm
- net MOSI: track 17.9 -> 22.0 mm, vias 1 -> 0
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
Commit message: PowerSwitch Layout near finish
Parts:
- added KK3: SK129, heatsink:SK129-HOLE
- added SJ2: (no value), jumper:SJ
- moved KK1 62.8 mm to (40.9, 81.4), turned to 90 degrees
- moved R42 58.0 mm to (42.8, 29.3), turned to 270 degrees
- moved R34 52.7 mm to (43.1, 42.9), turned to 270 degrees
- moved VR3 49.7 mm to (51.8, 20.7), turned to 180 degrees
- moved R35 45.9 mm to (52.2, 27.9), flipped to the top, turned to 90 degrees
- moved R30 44.8 mm to (48.6, 20.7)
- moved VR2 41.7 mm to (51.8, 20.7), flipped to the bottom, turned to 180 degrees
- moved VR9 39.3 mm to (38.1, 91.7), turned to 270 degrees
- moved Q6 36.1 mm to (48.0, 20.7), turned to 180 degrees
- moved R45 35.7 mm to (54.5, 27.9), flipped to the bottom
- moved R46 35.1 mm to (54.9, 20.7), flipped to the bottom
- moved D2 35.1 mm to (44.1, 20.7), flipped to the bottom, turned to 270 degrees
- moved VR1 32.4 mm to (57.5, 27.9), turned to 0 degrees
- moved D1 31.6 mm to (46.4, 20.7), flipped to the bottom, turned to 270 degrees
- moved R7 25.0 mm to (49.9, 27.9), flipped to the bottom, turned to 270 degrees
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Connections:
- net SW_AKT: now also SJ2.1
- net SW_KICK: now also SJ2.2
Routing:
- net +5V: track 51.0 -> 224.6 mm, vias 1 -> 7
- net SW_MOT: track 0.00 -> 134.7 mm, vias 0 -> 1
- net MOTION: track 0.00 -> 106.2 mm
- net SW_12V: track 0.00 -> 95.2 mm, vias 0 -> 3
- net SW_AKT: track 0.00 -> 84.6 mm, vias 0 -> 3
- net 24VIN: track 0.00 -> 77.8 mm
- net SW_BLAU: track 0.00 -> 77.7 mm, vias 0 -> 2
- net 12V-AKKU: track 0.00 -> 67.4 mm, vias 0 -> 3
- net DIV-24V: track 0.00 -> 62.3 mm
- net AKTUATOR: track 0.00 -> 62.2 mm
- net KICKER: track 0.00 -> 58.9 mm
- net 12V-EXT: track 0.00 -> 57.4 mm, vias 0 -> 2
- net 12V-I-OPV: track 0.00 -> 46.2 mm
- net 12V: track 22.0 -> 66.3 mm
- net N$49: track 0.00 -> 43.3 mm
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
Commit message: PowerSwitch Layout finished
Parts:
- removed KK2: SK104, heatsink:SK104
- removed KK3: SK129, heatsink:SK129-HOLE
- KK1: device heatsink:SK104 -> modifiedHeatsinks:SK104
- moved R_NULL_1 16.5 mm to (64.0, 11.3), flipped to the bottom, turned to 180 degrees
- moved R4 9.28 mm to (54.5, 13.3), turned to 180 degrees
- moved R_NULL_4 7.19 mm to (62.7, 18.2), flipped to the bottom, turned to 0 degrees
- moved R_NULL_2 6.48 mm to (62.7, 19.7), flipped to the bottom, turned to 0 degrees
- moved R_NULL_3 2.90 mm to (62.7, 22.2), turned to 0 degrees
- moved Q7 1.02 mm to (62.4, 27.9)
- moved VR1 0.76 mm to (58.3, 27.9)
- moved VR9 0.76 mm to (37.3, 91.7)
- moved R36 0.25 mm to (61.7, 64.6)
- moved R37 0.25 mm to (59.2, 64.6)
- moved R10 0.13 mm to (21.7, 58.5)
- moved R13 0.13 mm to (21.7, 60.8)
- moved R19 0.13 mm to (21.7, 63.1)
- moved R2 0.13 mm to (21.7, 56.3)
- moved R21 0.13 mm to (21.7, 60.8)
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Routing:
- net 12V: track 66.3 -> 131.6 mm, vias 0 -> 3
- net MOTION: track 106.2 -> 154.2 mm, vias 0 -> 1
- net AKTUATOR: track 62.2 -> 104.3 mm, vias 0 -> 2
- net KICKER: track 58.9 -> 100.1 mm, vias 0 -> 1
- net 12V-EXT: track 57.4 -> 86.0 mm, vias 2 -> 4
- net 12V-AKKU: track 67.4 -> 92.2 mm, vias 3 -> 4
- net SW_12V: track 95.2 -> 114.8 mm, vias 3 -> 4
- net SW_BLAU: track 77.7 -> 92.9 mm
- net SW_AKT: track 84.6 -> 97.9 mm
- net +5V: track 224.6 -> 233.9 mm
- net +3V3: track 77.7 -> 85.2 mm, vias 0 -> 1
- net LED_GRUEN: track 0.00 -> 5.38 mm
- net LED_ROT: track 0.00 -> 4.96 mm
- net LED_GELB: track 0.00 -> 4.96 mm
- net 12V-I-OPV: track 46.2 -> 42.9 mm
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