File: powerSwitch/pcb/CNC-PowerSwitch-2016-v0.95.sch (EAGLE design)
At the start: 102 parts, among them IC1 LM1458D, IC11 BTS6133, IC12 BTS6133, IC2 R-78E3.3-0.5, IC3 R-78E5.0-0.5, IC4 BTS555, P1 39-30-06_S, P4 39-30-06_S, P6 39-30-04_S, P8 39-30-04_S, Q1 16Mhz, Q2 IRF9530, Q3 IRF9530, Q4 IRF9530, Q5 IRF9530, T1 BC849, U2 TXB0108PWR

Commit message: powerswitch added ethernet, next step design
Parts:
- removed D3: ES1A, diode:GF1
- removed OK1: ILD213, optocoupler:ILD213
- removed R32: 1k, rcl:R-EU_R0805
- added C9: 1000µ/35V, rcl:CPOL-EUE5-10.5
- added D2: ES1A, diode:GF1
- added KK1, KK2: SK104, heatsink:SK104
- added Q6, Q7: BSS84, transistor-pnp:BC858ALT1SMD
- added R26, R7: 10k, rcl:R-EU_R0805
- added U$3, U$4, U$5, U$6: SK95-2M3, modifiedHeatsinks:SK95-2M3
- T1: value BC849 -> NX7002BK
Connections:
- removed net N$18: OK1A.EMIT, VR1.C
- removed net N$19: OK1A.C, OK1B.A
- removed net N$32: OK1B.EMIT, VR3.C
- removed net N$35: D1.C, D3.C, R32.2
- new net N$2: Q7.C, VR1.C
- new net N$8: Q6.C, VR3.C
- new net N$9: D2.A, R7.2
- net 12V: now also C9.+
- net 12V-AKKU: now also R7.1; no longer D3.A
- net 12V-EXT: now also R26.1; no longer D1.A
- net GND: now also C9.-, U2.GND
- net N$12: now also D1.A, R26.2; no longer OK1A.A, R32.1
- net N$30: now also Q6.E; no longer OK1B.COL
- net N$49: now also Q7.E; no longer OK1A.COL
- net SW_12V: now also D1.C, D2.C, Q6.B, Q7.B; no longer OK1B.C
Other:
- moved on the sheet: D1, Q2, Q3, Q4, Q5, R30, R34, R35, R42, R45, R46, VR1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

Commit message: PowerSwitch Layout near finish
Parts:
- added KK3: SK129, heatsink:SK129
- added SJ2: (no value), jumper:SJ
Connections:
- net SW_AKT: now also SJ2.1
- net SW_KICK: now also SJ2.2
Changed lines of the file:
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@@
 <part name="GND6" library="supply1" deviceset="GND" device=""/>
 <part name="GND8" library="supply1" deviceset="GND" device=""/>
+<part name="SJ2" library="jumper" deviceset="SJ" device=""/>
+<part name="KK3" library="heatsink" deviceset="SK129" device=""/>
 </parts>
 <sheets>
@@
 <instance part="C9" gate="G$1" x="114.3" y="88.9"/>
 <instance part="GND6" gate="1" x="114.3" y="78.74" rot="MR0"/>
+<instance part="SJ2" gate="1" x="27.94" y="114.3" rot="MR0"/>
+<instance part="KK3" gate="1" x="213.36" y="50.8"/>
 </instances>
 <busses>
@@
 <pinref part="VR7" gate="G$1" pin="A"/>
 </segment>
+<segment>
+<pinref part="SJ2" gate="1" pin="1"/>
+<wire x1="35.56" y1="114.3" x2="33.02" y2="114.3" width="0.1524" layer="91"/>
+<label x="35.56" y="114.3" size="1.27" layer="95" xref="yes"/>
+</segment>
 </net>
 <net name="SW_MOT" class="0">
@@
 <pinref part="VR8" gate="G$1" pin="A"/>
 </segment>
-</net>
+<segment>
+<pinref part="SJ2" gate="1" pin="2"/>
+<wire x1="20.32" y1="114.3" x2="22.86" y2="114.3" width="0.1524" layer="91"/>
+<label x="20.32" y="114.3" size="1.27" layer="95" rot="R180" xref="yes"/>
+</segment>
+</net>

Commit message: PowerSwitch Layout finished
Parts:
- removed KK2: SK104, heatsink:SK104
- removed KK3: SK129, heatsink:SK129
- KK1: device heatsink:SK104 -> modifiedHeatsinks:SK104
Changed lines of the file:
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@@
 <part name="R1" library="rcl" deviceset="R-EU_" device="R0805" value="560"/>
 <part name="3V3" library="led" deviceset="LED" device="CHIPLED_0805"/>
-<part name="KK1" library="heatsink" deviceset="SK104" device=""/>
-<part name="KK2" library="heatsink" deviceset="SK104" device=""/>
+<part name="KK1" library="modifiedHeatsinks" deviceset="SK104" device=""/>
 <part name="U$3" library="modifiedHeatsinks" deviceset="SK95-2M3" device=""/>
 <part name="U$4" library="modifiedHeatsinks" deviceset="SK95-2M3" device=""/>
@@
 <part name="GND8" library="supply1" deviceset="GND" device=""/>
 <part name="SJ2" library="jumper" deviceset="SJ" device=""/>
-<part name="KK3" library="heatsink" deviceset="SK129" device=""/>
 </parts>
 <sheets>
@@
 </instance>
 <instance part="KK1" gate="1" x="248.92" y="106.68" rot="R270"/>
-<instance part="KK2" gate="1" x="248.92" y="157.48" rot="R270"/>
 <instance part="U$3" gate="G$1" x="231.14" y="73.66"/>
 <instance part="U$4" gate="G$1" x="231.14" y="81.28"/>
@@
 <instance part="GND6" gate="1" x="114.3" y="78.74" rot="MR0"/>
 <instance part="SJ2" gate="1" x="27.94" y="114.3" rot="MR0"/>
-<instance part="KK3" gate="1" x="213.36" y="50.8"/>
 </instances>
 <busses>
