File: beagle2can/beagle2can.sch (EAGLE design)
At the start: 36 parts, among them IC1 R-785.0-0.5, P1 39-30-04_S, U1 TXB0108PWR

Commit message: beagle2can layout finished
Parts:
- U$1: device adafruit:BEAGLEBONE_OUTLINE -> ownParts:BEAGLEBONE_OUTLINE
Connections:
- net CON_24V: now also RJ_1.P$4, RJ_2.P$4
Changed lines of the file:
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@@
 <part name="C1" library="rcl" deviceset="CPOL-EU" device="D" value="47uF/35V"/>
 <part name="C2" library="rcl" deviceset="CPOL-EU" device="D" value="47uF/35V"/>
-<part name="U$1" library="adafruit" deviceset="BEAGLEBONE_OUTLINE" device=""/>
+<part name="U$1" library="ownParts" deviceset="BEAGLEBONE_OUTLINE" device=""/>
 <part name="P1" library="con-molex-mini-fit" deviceset="39-30-?04?_S" device=""/>
 <part name="P+1" library="supply1" deviceset="+5V" device=""/>
@@
 </segment>
 </net>
+<net name="CON_24V" class="0">
+<segment>
+<pinref part="RJ_1" gate="G$1" pin="P$4"/>
+<wire x1="33.02" y1="132.08" x2="40.64" y2="132.08" width="0.1524" layer="91"/>
+<label x="33.02" y="132.08" size="1.27" layer="95" rot="R180" xref="yes"/>
+</segment>
+<segment>
+<wire x1="121.92" y1="132.08" x2="129.54" y2="132.08" width="0.1524" layer="91"/>
+<label x="121.92" y="132.08" size="1.27" layer="95" rot="R180" xref="yes"/>
+<pinref part="RJ_2" gate="G$1" pin="P$4"/>
+</segment>
+</net>
