File: actuator/BBB_Cape/pcb/CN-Cape-1.1.brd (EAGLE design)
At the start: 160 x 86.4 mm, 108 parts, among them IC3 LM340MP-05, IC4 LM2576, IC5 LM2575, P8 BeagleBoard 2x23, P9 BeagleBoard 2x23, U1 ADUM1200ARZ, U2 ADUM1300ARWZ, U3 ADUM1200ARZ, U4 ADUM1300ARWZ

Commit message: little changes and part list for beagle2can, cape1.1
Parts:
- moved R29 1.27 mm to (145.8, 68.8)
- moved R12 0.25 mm to (130.0, 45.0)
Routing:
- net N$17: track 11.2 -> 9.95 mm
- net I2C2_SCL: track 50.0 -> 51.3 mm
Changed lines of the file:
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@@
 <?xml version="1.0" encoding="utf-8"?>
 <!DOCTYPE eagle SYSTEM "eagle.dtd">
-<eagle version="7.5.0">
+<eagle version="7.7.0">
 <drawing>
 <settings>
@@
 </class>
 </classes>
-<designrules name="qp_designrules_8mil">
+<designrules name="8mils">
 <description language="en">&lt;b&gt;EAGLE Design Rules&lt;/b&gt;
 &lt;p&gt;
@@
 <param name="layerSetup" value="(1*16)"/>
 <param name="mtCopper" value="0.035mm 0.035mm 0.035mm 0.035mm 0.035mm 0.035mm 0.035mm 0.035mm 0.035mm 0.035mm 0.035mm 0.035mm 0.035mm 0.035mm 0.035mm 0.035mm"/>
-<param name="mtIsolate" value="1.5mm 1.5mm 1.5mm 1.5mm 1.5mm 1.5mm 1.5mm 1.5mm 1.5mm 1.5mm 1.5mm 1.5mm 1.5mm 1.5mm 1.5mm"/>
+<param name="mtIsolate" value="1.5mm 0.15mm 0.2mm 0.15mm 0.2mm 0.15mm 0.2mm 0.15mm 0.2mm 0.15mm 0.2mm 0.15mm 0.2mm 0.15mm 0.2mm"/>
 <param name="mdWireWire" value="8mil"/>
 <param name="mdWirePad" value="8mil"/>
@@
 <param name="mdViaViaSameLayer" value="8mil"/>
 <param name="mnLayersViaInSmd" value="2"/>
-<param name="mdCopperDimension" value="20mil"/>
-<param name="mdDrill" value="20mil"/>
+<param name="mdCopperDimension" value="40mil"/>
+<param name="mdDrill" value="10mil"/>
 <param name="mdSmdStop" value="0mil"/>
 <param name="msWidth" value="8mil"/>
-<param name="msDrill" value="20mil"/>
-<param name="msMicroVia" value="0.1mm"/>
-<param name="msBlindViaRatio" value="0.5"/>
+<param name="msDrill" value="0.6mm"/>
+<param name="msMicroVia" value="0mil"/>
+<param name="msBlindViaRatio" value="0"/>
 <param name="rvPadTop" value="0.25"/>
 <param name="rvPadInner" value="0.25"/>
@@
 <param name="rvMicroViaOuter" value="0.25"/>
 <param name="rvMicroViaInner" value="0.25"/>
-<param name="rlMinPadTop" value="8mil"/>
+<param name="rlMinPadTop" value="10mil"/>
 <param name="rlMaxPadTop" value="20mil"/>
-<param name="rlMinPadInner" value="8mil"/>
+<param name="rlMinPadInner" value="10mil"/>
 <param name="rlMaxPadInner" value="20mil"/>
-<param name="rlMinPadBottom" value="8mil"/>
+<param name="rlMinPadBottom" value="10mil"/>
 <param name="rlMaxPadBottom" value="20mil"/>
 <param name="rlMinViaOuter" value="8mil"/>
@@
 <param name="rlMinViaInner" value="8mil"/>
 <param name="rlMaxViaInner" value="20mil"/>
-<param name="rlMinMicroViaOuter" value="0.35mm"/>
+<param name="rlMinMicroViaOuter" value="8mil"/>
 <param name="rlMaxMicroViaOuter" value="20mil"/>
-<param name="rlMinMicroViaInner" value="0.35mm"/>
+<param name="rlMinMicroViaInner" value="8mil"/>
 <param name="rlMaxMicroViaInner" value="20mil"/>
 <param name="psTop" value="-1"/>
@@
 <param name="mvStopFrame" value="0.1"/>
 <param name="mvCreamFrame" value="0"/>
-<param name="mlMinStopFrame" value="2mil"/>
-<param name="mlMaxStopFrame" value="2mil"/>
+<param name="mlMinStopFrame" value="0mil"/>
+<param name="mlMaxStopFrame" value="20mil"/>
 <param name="mlMinCreamFrame" value="0mil"/>
 <param name="mlMaxCreamFrame" value="0mil"/>
@@
 <element name="R27" library="rcl" package="R0805" value="10k" x="147.066" y="57.404"/>
 <element name="R28" library="rcl" package="R0805" value="10k" x="147.066" y="59.944"/>
-<element name="R29" library="rcl" package="R0805" value="330" x="145.796" y="67.564" rot="R90"/>
+<element name="R29" library="rcl" package="R0805" value="330" x="145.796" y="68.834" rot="R90"/>
 <element name="R30" library="rcl" package="R0805" value="330" x="138.43" y="63.754" rot="R90"/>
 <element name="CON_SPI-EXT" library="con-ml" package="ML6" value="" x="134.112" y="22.352" rot="MR0"/>
@@
 <element name="R10" library="rcl" package="R0805" value="10k" x="137.922" y="44.958" rot="R90"/>
 <element name="R11" library="rcl" package="R0805" value="10k" x="133.858" y="44.958" rot="R90"/>
-<element name="R12" library="rcl" package="R0805" value="10k" x="129.794" y="44.958" rot="R90"/>
+<element name="R12" library="rcl" package="R0805" value="10k" x="130.048" y="44.958" rot="R90"/>
 <element name="R31" library="rcl" package="R0805" value="10k" x="155.956" y="20.828" rot="R90"/>
 <element name="R32" library="rcl" package="R0805" value="10k" x="136.906" y="54.61" rot="MR90"/>
@@
 <wire x1="139.192" y1="57.404" x2="141.986" y2="57.404" width="0.254" layer="1"/>
 <wire x1="146.116" y1="57.404" x2="141.986" y2="57.404" width="0.254" layer="1"/>
-<wire x1="145.796" y1="66.614" x2="145.796" y2="63.5" width="0.254" layer="1"/>
+<wire x1="145.796" y1="67.884" x2="145.796" y2="63.5" width="0.254" layer="1"/>
 <via x="145.796" y="63.5" extent="1-16" drill="0.8"/>
 <wire x1="145.796" y1="63.5" x2="145.796" y2="58.928" width="0.254" layer="16"/>
@@
 <wire x1="129.794" y1="46.736" x2="129.794" y2="43.368" width="0.254" layer="16"/>
 <via x="129.794" y="46.736" extent="1-16" drill="0.6"/>
-<wire x1="129.794" y1="45.908" x2="129.794" y2="46.736" width="0.254" layer="1"/>
+<wire x1="130.048" y1="45.908" x2="129.794" y2="46.736" width="0.254" layer="1"/>
 </signal>
 <signal name="SW_BUNDLE-LED_3V">
@@
 <wire x1="145.034" y1="77.978" x2="145.034" y2="70.612" width="0.254" layer="1"/>
 <wire x1="145.034" y1="70.612" x2="145.796" y2="69.85" width="0.254" layer="1"/>
-<wire x1="145.796" y1="69.85" x2="145.796" y2="68.514" width="0.254" layer="1"/>
+<wire x1="145.796" y1="69.85" x2="145.796" y2="69.784" width="0.254" layer="1"/>
 </signal>
 <signal name="N$18">
@@
 <contactref element="PNP3" pad="B"/>
 <contactref element="R12" pad="1"/>
-<wire x1="129.794" y1="44.008" x2="129.794" y2="42.06" width="0.254" layer="1"/>
-<wire x1="129.794" y1="42.06" x2="128.712" y2="40.978" width="0.254" layer="1"/>
+<wire x1="130.048" y1="44.008" x2="130.048" y2="42.314" width="0.254" layer="1"/>
+<wire x1="130.048" y1="42.314" x2="128.712" y2="40.978" width="0.254" layer="1"/>
 </signal>
 <signal name="N$23">
