File: beagle2can/pcb/beagle2can.brd (EAGLE design)
At the start: 86.6 x 86.5 mm, 36 parts, among them IC1 R-785.0-0.5, P1 39-30-04?_S, U1 TXB0108PWR

Commit message: little changes and part list for beagle2can, cape1.1
Parts:
- moved C5 0.13 mm to (18.3, 45.3)
- moved C8 0.13 mm to (18.3, 43.3)
Connections:
- net GND: now also U$1.80
Changed lines of the file:
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@@
 </class>
 </classes>
-<designrules name="default">
-<description language="de">&lt;b&gt;EAGLE Design Rules&lt;/b&gt;
-&lt;p&gt;
-Die Standard-Design-Rules sind so gewählt, dass sie für
-die meisten Anwendungen passen. Sollte ihre Platine
-besondere Anforderungen haben, treffen Sie die erforderlichen
-Einstellungen hier und speichern die Design Rules unter
-einem neuen Namen ab.</description>
+<designrules name="8mils">
 <description language="en">&lt;b&gt;EAGLE Design Rules&lt;/b&gt;
 &lt;p&gt;
@@
 <param name="mnLayersViaInSmd" value="2"/>
 <param name="mdCopperDimension" value="40mil"/>
-<param name="mdDrill" value="8mil"/>
+<param name="mdDrill" value="10mil"/>
 <param name="mdSmdStop" value="0mil"/>
-<param name="msWidth" value="10mil"/>
-<param name="msDrill" value="24mil"/>
-<param name="msMicroVia" value="9.99mm"/>
-<param name="msBlindViaRatio" value="0.5"/>
+<param name="msWidth" value="8mil"/>
+<param name="msDrill" value="0.6mm"/>
+<param name="msMicroVia" value="0mil"/>
+<param name="msBlindViaRatio" value="0"/>
 <param name="rvPadTop" value="0.25"/>
 <param name="rvPadInner" value="0.25"/>
@@
 <param name="rlMinViaInner" value="8mil"/>
 <param name="rlMaxViaInner" value="20mil"/>
-<param name="rlMinMicroViaOuter" value="4mil"/>
+<param name="rlMinMicroViaOuter" value="8mil"/>
 <param name="rlMaxMicroViaOuter" value="20mil"/>
-<param name="rlMinMicroViaInner" value="4mil"/>
+<param name="rlMinMicroViaInner" value="8mil"/>
 <param name="rlMaxMicroViaInner" value="20mil"/>
 <param name="psTop" value="-1"/>
@@
 <param name="psElongationLong" value="100"/>
 <param name="psElongationOffset" value="100"/>
-<param name="mvStopFrame" value="1"/>
+<param name="mvStopFrame" value="0.1"/>
 <param name="mvCreamFrame" value="0"/>
-<param name="mlMinStopFrame" value="4mil"/>
-<param name="mlMaxStopFrame" value="4mil"/>
+<param name="mlMinStopFrame" value="0mil"/>
+<param name="mlMaxStopFrame" value="20mil"/>
 <param name="mlMinCreamFrame" value="0mil"/>
 <param name="mlMaxCreamFrame" value="0mil"/>
@@
 <element name="C3" library="rcl" package="C0603" value="100n" x="5.969" y="21.844" rot="MR180"/>
 <element name="C4" library="rcl" package="C0603" value="100n" x="5.969" y="9.398" rot="MR180"/>
-<element name="C5" library="rcl" package="C0603" value="100n" x="18.288" y="45.212"/>
+<element name="C5" library="rcl" package="C0603" value="100n" x="18.288" y="45.339"/>
 <element name="C6" library="rcl" package="C0603" value="100n" x="32.004" y="24.13"/>
 <element name="C7" library="rcl" package="C0603" value="100n" x="32.004" y="21.59"/>
-<element name="C8" library="rcl" package="C0603" value="100n" x="18.288" y="43.434"/>
+<element name="C8" library="rcl" package="C0603" value="100n" x="18.288" y="43.307"/>
 <element name="RJ_1" library="ownParts" package="RJ10" value="RJ10" x="10.414" y="14.859" rot="R270"/>
 <element name="RJ_2" library="ownParts" package="RJ10" value="RJ10" x="10.414" y="27.305" rot="R270"/>
@@
 <via x="20.447" y="44.323" extent="1-16" drill="0.4"/>
 <via x="22.098" y="42.926" extent="1-16" drill="0.4"/>
+<contactref element="U$1" pad="80"/>
 </signal>
 <signal name="SYS_5V">
@@
 <wire x1="3.683" y1="21.844" x2="6.604" y2="21.844" width="0.254" layer="1"/>
 <wire x1="7.493" y1="26.289" x2="6.604" y2="27.178" width="0.6096" layer="1"/>
-<wire x1="17.438" y1="43.434" x2="13.716" y2="43.434" width="0.4064" layer="1"/>
-<wire x1="13.716" y1="43.434" x2="13.208" y2="43.434" width="0.4064" layer="1"/>
-<wire x1="13.208" y1="43.434" x2="12.319" y2="44.323" width="0.4064" layer="1"/>
+<wire x1="13.843" y1="43.307" x2="13.335" y2="43.307" width="0.4064" layer="1"/>
+<wire x1="13.335" y1="43.307" x2="12.319" y2="44.323" width="0.4064" layer="1"/>
 <wire x1="16.002" y1="41.402" x2="16.002" y2="42.545" width="0.254" layer="16"/>
 <wire x1="16.002" y1="42.545" x2="15.748" y2="42.799" width="0.254" layer="16"/>
 <wire x1="15.748" y1="42.799" x2="14.351" y2="42.799" width="0.254" layer="16"/>
-<wire x1="14.351" y1="42.799" x2="13.716" y2="43.434" width="0.254" layer="16"/>
-<via x="13.716" y="43.434" extent="1-16" drill="0.4"/>
+<wire x1="14.351" y1="42.799" x2="13.843" y2="43.307" width="0.254" layer="16"/>
+<via x="13.843" y="43.307" extent="1-16" drill="0.4"/>
 <wire x1="11.049" y1="45.593" x2="12.319" y2="44.323" width="0.4064" layer="16"/>
 <wire x1="4.572" y1="75.184" x2="3.683" y2="74.295" width="0.8128" layer="16"/>
@@
 <wire x1="3.683" y1="44.323" x2="6.223" y2="41.783" width="0.8128" layer="1"/>
 <wire x1="11.049" y1="45.593" x2="3.683" y2="45.593" width="0.4064" layer="16"/>
+<wire x1="13.843" y1="43.307" x2="17.438" y2="43.307" width="0.4064" layer="1"/>
 </signal>
 <signal name="CAN0_RX">
@@
 <wire x1="16.891" y1="13.8335" x2="16.964" y2="13.9065" width="0.254" layer="16"/>
 <wire x1="5.334" y1="17.5768" x2="5.334" y2="17.018" width="0.254" layer="16"/>
-<wire x1="5.334" y1="17.018" x2="6.731" y2="15.621" width="0.254" layer="16"/>
-<wire x1="6.731" y1="15.621" x2="15.24" y2="15.621" width="0.254" layer="16"/>
-<wire x1="15.24" y1="15.621" x2="16.9545" y2="13.9065" width="0.254" layer="16"/>
+<wire x1="5.334" y1="17.018" x2="6.858" y2="15.494" width="0.254" layer="16"/>
+<wire x1="6.858" y1="15.494" x2="15.367" y2="15.494" width="0.254" layer="16"/>
+<wire x1="15.367" y1="15.494" x2="16.9545" y2="13.9065" width="0.254" layer="16"/>
 <wire x1="16.9545" y1="13.9065" x2="16.964" y2="13.9065" width="0.254" layer="16"/>
 </signal>
@@
 <wire x1="18.288" y1="14.5955" x2="19.504" y2="15.8115" width="0.254" layer="16"/>
 <wire x1="6.604" y1="17.5768" x2="6.604" y2="17.145" width="0.254" layer="16"/>
-<wire x1="6.604" y1="17.145" x2="7.62" y2="16.129" width="0.254" layer="16"/>
-<wire x1="7.62" y1="16.129" x2="15.494" y2="16.129" width="0.254" layer="16"/>
-<wire x1="15.494" y1="16.129" x2="16.256" y2="15.367" width="0.254" layer="16"/>
+<wire x1="6.604" y1="17.145" x2="7.747" y2="16.002" width="0.254" layer="16"/>
+<wire x1="7.747" y1="16.002" x2="15.621" y2="16.002" width="0.254" layer="16"/>
+<wire x1="15.621" y1="16.002" x2="16.256" y2="15.367" width="0.254" layer="16"/>
 <wire x1="16.256" y1="15.367" x2="17.5165" y2="15.367" width="0.254" layer="16"/>
 <wire x1="17.5165" y1="15.367" x2="18.288" y2="14.5955" width="0.254" layer="16"/>
@@
 <wire x1="16.891" y1="26.2795" x2="16.964" y2="26.3525" width="0.254" layer="16"/>
 <wire x1="5.334" y1="30.0228" x2="5.334" y2="29.591" width="0.254" layer="16"/>
-<wire x1="5.334" y1="29.591" x2="6.604" y2="28.321" width="0.254" layer="16"/>
-<wire x1="6.604" y1="28.321" x2="14.9955" y2="28.321" width="0.254" layer="16"/>
-<wire x1="14.9955" y1="28.321" x2="16.964" y2="26.3525" width="0.254" layer="16"/>
+<wire x1="5.334" y1="29.591" x2="7.366" y2="27.559" width="0.254" layer="16"/>
+<wire x1="7.366" y1="27.559" x2="15.7575" y2="27.559" width="0.254" layer="16"/>
+<wire x1="15.7575" y1="27.559" x2="16.964" y2="26.3525" width="0.254" layer="16"/>
 </signal>
 <signal name="CAN1_H">
@@
 <wire x1="18.415" y1="27.1685" x2="19.504" y2="28.2575" width="0.254" layer="16"/>
 <wire x1="6.604" y1="30.0228" x2="6.604" y2="29.591" width="0.254" layer="16"/>
-<wire x1="6.604" y1="29.591" x2="7.366" y2="28.829" width="0.254" layer="16"/>
-<wire x1="7.366" y1="28.829" x2="15.24" y2="28.829" width="0.254" layer="16"/>
-<wire x1="15.24" y1="28.829" x2="16.002" y2="28.067" width="0.254" layer="16"/>
-<wire x1="16.002" y1="28.067" x2="17.5165" y2="28.067" width="0.254" layer="16"/>
+<wire x1="6.604" y1="29.591" x2="8.128" y2="28.067" width="0.254" layer="16"/>
 <wire x1="17.5165" y1="28.067" x2="18.415" y2="27.1685" width="0.254" layer="16"/>
+<wire x1="8.128" y1="28.067" x2="17.5165" y2="28.067" width="0.254" layer="16"/>
 </signal>
 <signal name="CAN0_TX_5V">
@@
 <wire x1="29.083" y1="34.798" x2="29.083" y2="45.085" width="0.4064" layer="16"/>
 <wire x1="29.083" y1="45.085" x2="28.448" y2="45.72" width="0.4064" layer="16"/>
-<wire x1="17.438" y1="45.212" x2="16.51" y2="45.212" width="0.254" layer="1"/>
-<wire x1="16.51" y1="45.212" x2="16.002" y2="45.72" width="0.254" layer="1"/>
 <via x="16.002" y="45.72" extent="1-16" drill="0.4"/>
 <wire x1="16.002" y1="45.72" x2="16.002" y2="47.244" width="0.254" layer="16"/>
@@
 <wire x1="26.797" y1="21.59" x2="28.321" y2="21.59" width="0.4064" layer="16"/>
 <wire x1="28.321" y1="21.59" x2="29.083" y2="22.352" width="0.4064" layer="16"/>
+<wire x1="16.002" y1="45.72" x2="16.383" y2="45.339" width="0.4064" layer="1"/>
+<wire x1="16.383" y1="45.339" x2="17.438" y2="45.339" width="0.4064" layer="1"/>
 </signal>
 <signal name="I2C1_SCL">
