File: beagle2can/pcb/beagle2can.sch (EAGLE design)
At the start: 36 parts, among them IC1 R-785.0-0.5, P1 39-30-04_S, U1 TXB0108PWR

Commit message: little changes and part list for beagle2can, cape1.1
Connections:
- net GND: now also U$1.GNDA_ADC
Changed lines of the file:
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@@
 <wire x1="215.9" y1="38.1" x2="215.9" y2="35.56" width="0.1524" layer="91"/>
 <pinref part="GND7" gate="1" pin="GND"/>
+<pinref part="U$1" gate="G$1" pin="GNDA_ADC"/>
+<wire x1="208.28" y1="50.8" x2="215.9" y2="50.8" width="0.1524" layer="91"/>
+<wire x1="215.9" y1="50.8" x2="215.9" y2="38.1" width="0.1524" layer="91"/>
+<junction x="215.9" y="38.1"/>
 </segment>
 <segment>
