File: kicker/rekick2017/pcb/rekick2017-v0.1.brd (EAGLE design)
At the start: 160 x 100 mm, 195 parts, among them IC1 74LVC1G02GW, IC2 4043D, IC3 LM1117, IC4 LM1458D, P1 39-30-06?_S, P2 39-30-08?_S, Q1 16MHz, Q2 IKW 25N120, Q3 PSMN7R8-120PS, Q4 PSMN7R8-120PS, Q5 IPD90P04P4L, Q6 IRF840, T1 BC859, T2 BC849, T3 BC849, T4 BC849, T5 IRLML6344TRPBF, U1 TXB0108PWR, U4 LM2675, U5 ADUM4190BRIZ

Commit message: Kicker - Layout halb fertig
Parts:
- removed C20: 47µ/35V, rcl:PANASONIC_D
- removed C22: 10n/35V, rcl:C0603
- removed CAP_0V, CAP_330V, COIL_IN, COIL_OUT: WIREPADSMD5-5, mywirepad:5-5
- removed D7: ES1A, diode:SMA-DO214AC
- removed L6: 150µH, Inductor-Fastron:PISM
- removed LED2, LED3: (no value), led:CHIP-LED0805
- removed R35: 4.7k, rcl:R0805
- removed R38: 5.6k, rcl:R0805
- removed R40, R41: 1k, rcl:R0805
- removed U$16, U$8: DCDC_OKI-78SRVERTICAL, carrilib:OKI-78SRV
- removed VR2, VR3: TL431_SOT23, 1_USER:SOT23
- added D6: ES1A, diode:SMA-DO214AC
- added H5: MOUNT-PAD-ROUND3.0, holes:3,0-PAD
- added KK2: SK104, heatsink:SK104
- added U2: R-7805, recom-intl:R-78XX
- added U3: R-7812, recom-intl:R-78XX
- Q2: value IKW 25N120 -> IKW40N120T2FKSA1
- U4: value LM2675 -> R-7805; device LM2675M-3.3:SOIC127P620X175-8N -> recom-intl:R-78XX
- moved U4 133.5 mm to (25.7, 89.4), flipped to the top, turned to 0 degrees
- moved LED10 94.7 mm to (157.7, 34.3), turned to 270 degrees
- moved R59 89.2 mm to (157.2, 15.7), flipped to the bottom, turned to 270 degrees
- moved D13 79.9 mm to (150.9, 15.5), flipped to the bottom, turned to 90 degrees
- moved R57 71.0 mm to (131.7, 6.86), flipped to the bottom, turned to 0 degrees
- moved R43 68.5 mm to (131.7, 8.89), flipped to the bottom, turned to 180 degrees
- moved T3 66.4 mm to (131.7, 11.9), flipped to the bottom, turned to 90 degrees
- moved LED9 64.2 mm to (158.1, 61.6)
- moved R24 64.1 mm to (125.5, 11.0), flipped to the bottom, turned to 180 degrees
- moved C34 51.0 mm to (63.2, 53.7), turned to 90 degrees
- moved R44 49.2 mm to (114.9, 8.89), flipped to the bottom, turned to 180 degrees
- moved C37 49.0 mm to (79.4, 49.3), turned to 90 degrees
- moved C39 46.2 mm to (81.4, 49.3), turned to 90 degrees
- moved LED11 46.2 mm to (106.9, 2.29)
- moved LED5 45.7 mm to (109.0, 2.29)
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Connections:
- removed net N$26: C22.2, D7.K, L6.2, U4.8
- removed net N$33: C22.1, U4.1
- removed net N$61: R35.1, R38.2, VR3.2
- removed net N$62: LED2.C, VR2.1
- removed net N$63: LED3.C, VR3.1
- removed net N$65: LED2.A, R40.1
- removed net N$66: LED3.A, R41.1
- new net N$1: R29.1, U$2.27
- net +12V: now also U3.3; no longer L6.1, U4.4
- net +24V: now also U2.1, U3.1, U4.1; no longer C20.+, U$16.1, U$8.1, U4.7
- net +5V: now also U2.3; no longer R40.2, R41.2, U$16.3
- net +5V/1: now also U4.3; no longer U$8.3
- net ADC_CAP: no longer R35.2, VR2.2
- net CAP_0V: no longer CAP_0V.P$1
- net CAP_330V: no longer CAP_330V.P$1, COIL_OUT.P$1
- net CHARGE: now also D6.A; no longer U$2.22
- net COIL: no longer COIL_IN.P$1
- net GND: now also U2.2, U3.2, U4.2; no longer C20.-, D7.A, R38.1, U$16.2, U$8.2, U4.6, VR2.3, VR3.3
- net N$25: now also D6.K, U$2.22; no longer R29.1, U$2.16
Routing:
- net N$8: track 0.00 -> 169.7 mm, vias 0 -> 11
- net +24V: track 0.00 -> 94.8 mm
- net CAP_330V: track 0.00 -> 92.9 mm
- net +5V: track 0.00 -> 90.7 mm, vias 0 -> 4
- net +12V: track 0.00 -> 86.6 mm, vias 0 -> 4
- net GND1: track 0.00 -> 83.3 mm, vias 0 -> 2
- net N$39: track 0.00 -> 61.7 mm
- net N$76: track 0.00 -> 61.5 mm, vias 0 -> 1
- net N$17: track 0.00 -> 58.3 mm, vias 0 -> 2
- net N$58: track 0.00 -> 55.8 mm, vias 0 -> 1
- net CAP_+12V: track 0.00 -> 43.9 mm
- net N$44: track 0.00 -> 36.0 mm
- net COIL: track 0.00 -> 35.0 mm
- net ACTIVATE_BOOSTER: track 0.00 -> 33.2 mm
- net N$1: track 32.8 -> 0.00 mm
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- added copper zone on layer 1, net CAP_0V
- added copper zone on layer 16, net CAP_0V
- added copper zone on layer 1, net CAP_330V
- added copper zone on layer 16, net CAP_330V
- added copper zone on layer 1, net GND
- added copper zone on layer 16, net GND
- added copper zone on layer 1, net GND1
- added copper zone on layer 16, net GND1

Commit message: Kicker 2017
Parts:
- removed H5: MOUNT-PAD-ROUND3.0, holes:3,0-PAD
- IC1: value 74LVC1G02GW -> MC74VHC1G03
- KK1: device heatsink:SK104 -> ownParts:SK104
- moved R31 62.7 mm to (95.2, 14.1), turned to 0 degrees
- moved R50 60.6 mm to (95.2, 12.1), turned to 180 degrees
- moved C34 56.4 mm to (26.9, 10.5)
- moved R69 30.9 mm to (85.2, 37.8), turned to 180 degrees
- moved R55 26.7 mm to (77.1, 49.3)
- moved C28 25.5 mm to (5.33, 31.4), turned to 180 degrees
- moved R29 25.5 mm to (72.6, 61.5), turned to 0 degrees
- moved D4 24.4 mm to (72.6, 63.8), turned to 180 degrees
- moved C45 23.9 mm to (63.6, 65.0), flipped to the bottom, turned to 270 degrees
- moved U$1 23.4 mm to (5.33, 27.6), turned to 180 degrees
- moved R58 23.3 mm to (63.6, 68.3)
- moved IC2 22.5 mm to (63.6, 61.8)
- moved R45 22.5 mm to (18.0, 68.3)
- moved LED7 22.4 mm to (12.8, 68.3)
- moved R1 22.4 mm to (5.33, 23.5), turned to 180 degrees
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Connections:
- net !DONE: now also U$2.23; no longer U$2.25
- net KICK: now also U$2.25; no longer U$2.23
Routing:
- net +24V: track 94.8 -> 216.9 mm, vias 0 -> 1
- net +5V: track 90.7 -> 164.9 mm, vias 4 -> 11
- net MOSI: track 0.00 -> 54.0 mm
- net MISO: track 0.00 -> 52.2 mm
- net OC0A/MOSI_A: track 0.00 -> 49.7 mm, vias 0 -> 1
- net RST: track 0.00 -> 48.4 mm, vias 0 -> 1
- net NOTAUS: track 0.00 -> 39.5 mm, vias 0 -> 2
- net OC1A_FREQ/MISO_A: track 0.00 -> 38.6 mm, vias 0 -> 1
- net +3V3: track 0.00 -> 36.7 mm, vias 0 -> 2
- net RESET_NOTAUS: track 0.00 -> 32.2 mm, vias 0 -> 2
- net ÜBERSPANNUNG: track 0.00 -> 30.3 mm, vias 0 -> 3
- net ADC_CAP: track 8.54 -> 37.1 mm, vias 0 -> 1
- net SCK: track 0.00 -> 24.3 mm
- net CS_ETH: track 0.00 -> 23.0 mm
- net +5V/1: track 0.00 -> 21.6 mm
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
Commit message: rekick2017 final version?
Parts:
- moved C3 62.6 mm to (23.6, 22.4), turned to 270 degrees
- moved C40 62.3 mm to (6.22, 22.6), turned to 90 degrees
- moved U4 62.1 mm to (16.4, 22.5), turned to 90 degrees
- moved R47 38.1 mm to (8.51, 35.3)
- moved JP3 38.1 mm to (9.53, 35.8)
- moved JP4 38.1 mm to (19.4, 35.8)
- moved R16 38.1 mm to (8.51, 33.0)
- moved R7 38.1 mm to (8.51, 30.7)
- moved T5 38.1 mm to (8.51, 38.5)
- moved LED7 38.1 mm to (7.11, 30.6)
- moved R45 38.1 mm to (12.3, 30.6)
- moved R8 35.5 mm to (23.9, 33.3), turned to 0 degrees
- moved R70 32.9 mm to (85.2, 30.4), turned to 0 degrees
- moved T1 27.6 mm to (85.2, 34.2), turned to 0 degrees
- moved C34 25.2 mm to (30.9, 35.4), flipped to the bottom, turned to 180 degrees
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Routing:
- net +5V: track 164.9 -> 352.5 mm, vias 11 -> 16
- net ADC_24V_LOGIK/SCK_A: track 7.86 -> 92.9 mm, vias 1 -> 3
- net SERVO_PWM: track 0.00 -> 76.6 mm, vias 0 -> 1
- net TRIGGER_NOTAUS: track 8.71 -> 84.4 mm
- net ACTIVATE_SERVO: track 0.00 -> 74.7 mm, vias 0 -> 3
- net NOTAUS: track 39.5 -> 112.6 mm, vias 2 -> 4
- net CAN_RX: track 5.91 -> 77.6 mm, vias 0 -> 1
- net CAN_TX: track 3.20 -> 71.7 mm, vias 0 -> 1
- net ACTIVATE_BOOSTER: track 25.0 -> 70.0 mm, vias 0 -> 1
- net INT_ETH: track 20.9 -> 61.9 mm, vias 0 -> 2
- net RST_ETH: track 18.2 -> 57.4 mm, vias 0 -> 2
- net SCK: track 24.3 -> 62.8 mm
- net CS_ETH: track 23.0 -> 61.4 mm
- net ADC_24V_BOOSTER: track 10.6 -> 36.0 mm
- net CHARGE: track 10.2 -> 31.7 mm, vias 0 -> 1
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
Commit message: kicker2017final
Parts:
- removed R3, R74: 3.6, rcl:R2010
- removed T3: BC849, transistor:SOT23
- added R34: 50k, rcl:R0805
- added R36, R37, R38, R39: (no value), rcl:R1210
- added T6: (no value), zetex:SOT-23
- C10, C12, C30, C31, C35, C50, C51, C9: value 10µ/50V -> 10µ/35V
- LED11: device led:CHIPLED_0603 -> led:CHIP-LED0805
- R42: value 680 -> 1k
- T2, T4: value BC849 -> (none); device transistor:SOT23 -> zetex:SOT-23
- moved C44 0.25 mm to (88.3, 74.9)
- moved C57 0.25 mm to (77.5, 29.2)
- moved C14 0.25 mm to (92.3, 74.9)
- moved C59 0.25 mm to (73.4, 29.2)
- moved R61 0.18 mm to (116.7, 21.3)
- moved C4 0.13 mm to (75.6, 30.6)
- moved C5 0.13 mm to (71.4, 30.6)
- moved R62 0.13 mm to (116.7, 19.2)
- moved T4 0.13 mm to (85.2, 76.3), turned to 180 degrees
- turned T2 to 180 degrees
Connections:
- removed net N$58: Q3.D, Q4.D, R3.2, R61.1, R62.1, R74.2, U$3.10, U$3.11, U$3.12, U$3.9
- new net N$26: Q3.D, Q4.D, R36.2, R37.2, R38.2, R39.2, R61.1, R62.1, U$3.10, U$3.11, U$3.12, U$3.9
- net GND1: now also R34.1, T6.2; no longer T3.2
- net N$39: now also T4.1; no longer T4.3
- net N$45: now also T2.1; no longer T2.3
- net N$46: now also T4.3; no longer T4.1
- net N$47: now also T2.3; no longer T2.1
- net N$55: now also T6.1; no longer T3.3
- net N$56: now also R34.2, T6.3; no longer T3.1
- net N$86: now also R36.1, R37.1, R38.1, R39.1; no longer R3.1, R74.1
Routing:
- net N$26: track 0.00 -> 61.9 mm, vias 0 -> 1
- net N$58: track 55.8 -> 0.00 mm, vias 1 -> 0
- net GND1: track 83.3 -> 90.4 mm, vias 2 -> 3
- net N$86: track 8.29 -> 14.7 mm
- net +5V: track 352.5 -> 349.2 mm, vias 16 -> 15
- net N$56: track 4.20 -> 6.42 mm
- net ADC_CAP: track 37.1 -> 38.0 mm
- net N$78: track 31.5 -> 32.2 mm
- net GND: vias 5 -> 23
