File: kicker/rekick2017/pcb/rekick2017-v0.1.sch (EAGLE design)
At the start: 195 parts, among them IC1 74LVC1G02GW, IC2 4043D, IC3 LM1117, IC4 LM1458D, P1 39-30-06_S, P2 39-30-08_S, Q1 16MHz, Q2 IKW 25N120, Q3 PSMN7R8-120PS, Q4 PSMN7R8-120PS, Q5 IPD90P04P4L, Q6 IRF840, T1 BC859, T2 BC849, T3 BC849, T4 BC849, T5 IRLML6344TRPBF, U1 TXB0108PWR, U4 LM2675, U5 ADUM4190BRIZ

Commit message: Kicker - Layout halb fertig
Parts:
- removed C20: 47µ/35V, rcl:CPOL-EUD
- removed C22: 10n/35V, rcl:C-EUC0603
- removed CAP_0V, CAP_330V, COIL_IN, COIL_OUT: WIREPADSMD5-5, mywirepad:WIREPADSMD5-5
- removed D7: ES1A, diode:GF1
- removed L6: 150µH, Inductor-Fastron:L-EUPISM
- removed LED2, LED3: (no value), led:LEDCHIP-LED0805
- removed R35: 4.7k, rcl:R-EU_R0805
- removed R38: 5.6k, rcl:R-EU_R0805
- removed R40, R41: 1k, rcl:R-EU_R0805
- removed U$16, U$8: DCDC_OKI-78SRVERTICAL, carrilib:DCDC_OKI-78SRVERTICAL
- removed VR2, VR3: TL431_SOT23, 1_USER:TL431_SOT23
- added D6: ES1A, diode:GF1
- added H5: MOUNT-PAD-ROUND3.0, holes:MOUNT-PAD-ROUND3.0
- added KK2: SK104, heatsink:SK104
- added U2: R-7805, recom-intl:R-78XX
- added U3: R-7812, recom-intl:R-78XX
- Q2: value IKW 25N120 -> IKW40N120T2FKSA1
- U4: value LM2675 -> R-7805; device LM2675M-3.3:LM2675M-3.3 -> recom-intl:R-78XX
Connections:
- removed net N$26: C22.2, D7.C, L6.2, U4.VSW
- removed net N$33: C22.1, U4.CB
- removed net N$61: R35.1, R38.2, VR3.R
- removed net N$62: LED2.C, VR2.C
- removed net N$63: LED3.C, VR3.C
- removed net N$65: LED2.A, R40.1
- removed net N$66: LED3.A, R41.1
- new net N$1: R29.1, U$2.PB6
- net +12V: now also U3.OUT; no longer L6.1, U4.FB
- net +24V: now also U2.IN, U3.IN, U4.IN; no longer C20.+, U$16.VI, U$8.VI, U4.VIN
- net +5V: now also U2.OUT; no longer R40.2, R41.2, U$16.VO
- net +5V/1: now also U4.OUT; no longer U$8.VO
- net ADC_CAP: no longer R35.2, VR2.R
- net CAP_0V: no longer CAP_0V.P
- net CAP_330V: no longer CAP_330V.P, COIL_OUT.P
- net CHARGE: now also D6.A; no longer U$2.PC6
- net COIL: no longer COIL_IN.P
- net GND: now also U2.GND, U3.GND; no longer C20.-, D7.A, R38.1, U$16.GND, U$8.GND, VR2.A, VR3.A
- net N$25: now also D6.C, U$2.PC6; no longer R29.1, U$2.PB2
Other:
- moved on the sheet: C17, C18, C21, C3, C40, D4, LED5, LED6, LED7, R20, R29, R43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

Commit message: Kicker 2017
Parts:
- removed H5: MOUNT-PAD-ROUND3.0, holes:MOUNT-PAD-ROUND3.0
- IC1: value 74LVC1G02GW -> MC74VHC1G03
- KK1: device heatsink:SK104 -> ownParts:SK104
Connections:
- net !DONE: now also U$2.PB3; no longer U$2.PC7
- net KICK: now also U$2.PC7; no longer U$2.PB3
Changed lines of the file:
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@@
 <layer number="54" name="bGND_GNDA" color="1" fill="9" visible="no" active="no"/>
 <layer number="56" name="wert" color="7" fill="1" visible="no" active="no"/>
+<layer number="57" name="tCAD" color="7" fill="1" visible="no" active="no"/>
+<layer number="59" name="tCarbon" color="7" fill="1" visible="no" active="no"/>
+<layer number="60" name="bCarbon" color="7" fill="1" visible="no" active="no"/>
 <layer number="90" name="Modules" color="5" fill="1" visible="yes" active="yes"/>
 <layer number="91" name="Nets" color="2" fill="1" visible="yes" active="yes"/>
@@
 <layer number="109" name="fp9" color="12" fill="8" visible="no" active="no"/>
 <layer number="110" name="fp0" color="13" fill="8" visible="no" active="no"/>
+<layer number="111" name="LPC17xx" color="7" fill="1" visible="no" active="yes"/>
+<layer number="112" name="tSilk" color="7" fill="1" visible="no" active="yes"/>
+<layer number="113" name="ReferenceLS" color="7" fill="1" visible="no" active="no"/>
 <layer number="116" name="Patch_BOT" color="9" fill="4" visible="yes" active="yes"/>
 <layer number="118" name="Rect_Pads" color="4" fill="1" visible="no" active="no"/>
@@
 <layer number="124" name="bTestmark" color="3" fill="3" visible="no" active="no"/>
 <layer number="125" name="_tNames" color="7" fill="1" visible="no" active="yes"/>
+<layer number="126" name="_bNames" color="7" fill="1" visible="no" active="yes"/>
+<layer number="127" name="_tValues" color="7" fill="1" visible="no" active="yes"/>
+<layer number="128" name="_bValues" color="7" fill="1" visible="no" active="yes"/>
+<layer number="129" name="Mask" color="7" fill="1" visible="yes" active="yes"/>
 <layer number="131" name="tAdjust" color="15" fill="1" visible="no" active="no"/>
 <layer number="132" name="bAdjust" color="5" fill="1" visible="no" active="no"/>
 <layer number="144" name="Drill_legend" color="7" fill="1" visible="no" active="yes"/>
+<layer number="150" name="Notes" color="7" fill="1" visible="no" active="yes"/>
 <layer number="151" name="HeatSink" color="7" fill="1" visible="yes" active="yes"/>
+<layer number="152" name="_bDocu" color="7" fill="1" visible="no" active="yes"/>
+<layer number="153" name="FabDoc1" color="6" fill="1" visible="no" active="no"/>
+<layer number="154" name="FabDoc2" color="2" fill="1" visible="no" active="no"/>
+<layer number="155" name="FabDoc3" color="7" fill="15" visible="no" active="no"/>
+<layer number="199" name="Contour" color="7" fill="1" visible="no" active="yes"/>
 <layer number="200" name="200bmp" color="1" fill="10" visible="no" active="no"/>
 <layer number="201" name="201bmp" color="2" fill="1" visible="no" active="no"/>
@@
 <layer number="223" name="223bmp" color="24" fill="1" visible="no" active="no"/>
 <layer number="224" name="224bmp" color="25" fill="1" visible="no" active="no"/>
+<layer number="225" name="225bmp" color="7" fill="1" visible="yes" active="yes"/>
+<layer number="226" name="226bmp" color="7" fill="1" visible="yes" active="yes"/>
+<layer number="227" name="227bmp" color="7" fill="1" visible="yes" active="yes"/>
+<layer number="228" name="228bmp" color="7" fill="1" visible="yes" active="yes"/>
+<layer number="229" name="229bmp" color="7" fill="1" visible="yes" active="yes"/>
+<layer number="230" name="230bmp" color="7" fill="1" visible="yes" active="yes"/>
+<layer number="231" name="Eagle3D_PG1" color="7" fill="1" visible="no" active="no"/>
+<layer number="232" name="Eagle3D_PG2" color="7" fill="1" visible="no" active="no"/>
+<layer number="233" name="Eagle3D_PG3" color="7" fill="1" visible="no" active="no"/>
+<layer number="248" name="Housing" color="7" fill="1" visible="no" active="yes"/>
+<layer number="249" name="Edge" color="7" fill="1" visible="no" active="yes"/>
 <layer number="250" name="Descript" color="3" fill="1" visible="no" active="no"/>
 <layer number="251" name="SMDround" color="12" fill="11" visible="no" active="no"/>
 <layer number="254" name="OrgLBR" color="7" fill="1" visible="yes" active="yes"/>
+<layer number="255" name="routoute" color="7" fill="1" visible="yes" active="yes"/>
 </layers>
 <schematic xreflabel="%F%N/%S.%C%R" xrefpart="/%S.%C%R">
@@
 <part name="D3" library="diode" deviceset="BZX84CSMD" device="" value="SMD ZD 12"/>
 <part name="R11" library="rcl" deviceset="R-EU_" device="R0805" value="50k"/>
-<part name="IC1" library="74xx-little-de" deviceset="74*1G02" device="DBV" technology="AHC" value=" 74LVC1G02GW"/>
+<part name="IC1" library="74xx-little-de" deviceset="74*1G02" device="DBV" technology="AHC" value="MC74VHC1G03"/>
 <part name="R12" library="rcl" deviceset="R-EU_" device="R0805" value="1k"/>
 <part name="P+18" library="supply1" deviceset="+5V" device=""/>
@@
 <part name="R73" library="R2818" deviceset="R2818" device="" value="10m"/>
 <part name="Q4" library="transistor-power" deviceset="PMOSFET_N" device="TO220BV" value="PSMN7R8-120PS"/>
-<part name="KK1" library="heatsink" deviceset="SK104" device=""/>
+<part name="KK1" library="ownParts" deviceset="SK104" device=""/>
 <part name="R74" library="rcl" deviceset="R-EU_" device="R2010" value="3.6"/>
 <part name="C41" library="rcl" deviceset="C-EU" device="C1206" value="22n"/>
@@
 <part name="GND13" library="supply1" deviceset="GND" device=""/>
 <part name="GND15" library="supply1" deviceset="GND" device=""/>
-<part name="H5" library="holes" deviceset="MOUNT-PAD-ROUND" device="3.0"/>
 <part name="D6" library="diode" deviceset="GF1" device="" value="ES1A"/>
 </parts>
@@
 <instance part="GND13" gate="1" x="33.02" y="63.5"/>
 <instance part="GND15" gate="1" x="33.02" y="99.06"/>
-<instance part="H5" gate="G$1" x="238.76" y="109.22"/>
 </instances>
 <busses>
@@
 <net name="KICK" class="0">
 <segment>
-<pinref part="U$2" gate="G$1" pin="PB3"/>
-<wire x1="124.46" y1="137.16" x2="134.62" y2="137.16" width="0.1524" layer="91"/>
-<label x="134.62" y="137.16" size="1.27" layer="95" xref="yes"/>
+<wire x1="124.46" y1="124.46" x2="157.48" y2="124.46" width="0.1524" layer="91"/>
+<label x="157.48" y="124.46" size="1.27" layer="95" xref="yes"/>
+<pinref part="U$2" gate="G$1" pin="PC7"/>
 </segment>
 </net>
@@
 <net name="!DONE" class="0">
 <segment>
-<pinref part="U$2" gate="G$1" pin="PC7"/>
-<wire x1="157.48" y1="124.46" x2="124.46" y2="124.46" width="0.1524" layer="91"/>
-<label x="157.48" y="124.46" size="1.27" layer="95" xref="yes"/>
-</segment>
-</net>
+<wire x1="157.48" y1="137.16" x2="124.46" y2="137.16" width="0.1524" layer="91"/>
+<label x="157.48" y="137.16" size="1.27" layer="95" xref="yes"/>
+<pinref part="U$2" gate="G$1" pin="PB3"/>
+</segment>
+</net>

Commit message: kicker2017final
Parts:
- removed R3, R74: 3.6, rcl:R-EU_R2010
- removed T3: BC849, transistor:BC849
- added R34: 50k, rcl:R-EU_R0805
- added R36, R37, R38, R39: (no value), rcl:R-EU_R1210
- added T6: (no value), zetex:NMOSSOT23
- C10, C12, C30, C31, C35, C50, C51, C9: value 10µ/50V -> 10µ/35V
- LED11: device led:LEDCHIPLED_0603 -> led:LEDCHIP-LED0805
- R42: value 680 -> 1k
- T2, T4: value BC849 -> (none); device transistor:BC849 -> zetex:NMOSSOT23
Connections:
- removed net N$58: Q3.D, Q4.D, R3.2, R61.1, R62.1, R74.2, U$3.W12, U$3.W22, U$3.W32, U$3.W42
- new net N$26: Q3.D, Q4.D, R36.2, R37.2, R38.2, R39.2, R61.1, R62.1, U$3.W12, U$3.W22, U$3.W32, U$3.W42
- net CAP_0V: now also T4.S; no longer T4.E
- net GND: now also T2.S; no longer T2.E
- net GND1: now also R34.1, T6.S; no longer T3.E
- net N$39: now also T4.D; no longer T4.C
- net N$45: now also T2.D; no longer T2.C
- net N$46: now also T4.G; no longer T4.B
- net N$47: now also T2.G; no longer T2.B
- net N$55: now also T6.D; no longer T3.C
- net N$56: now also R34.2, T6.G; no longer T3.B
- net N$86: now also R36.1, R37.1, R38.1, R39.1; no longer R3.1, R74.1
Other:
- moved on the sheet: C10, C35, C50, C51, C52, C55, C56, R24
