File: kicker/rekick2017/pcb/rekick2017-v0.2.brd (EAGLE design)
At the start: 160 x 100 mm, 184 parts, among them IC1 SN74LVC1G02DBVR, IC2 4043D, IC3 LM1117, IC4 MCP602-I/SN, P1 39-30-06?_S, P2 39-30-08?_S, Q1 16MHz, Q2 IKW40N120T2FKSA1, Q3 PSMN7R8-120PS, Q4 PSMN7R8-120PS, Q5 IPD90P04P4L, Q6 IRF840, T1 BC859, T5 IRLML6344TRPBF, U1 TXB0108PWR, U2 R-7805, U3 R-7812, U4 R-7805, U5 ADUM4190BRIZ

Commit message: rekick2017 0.2 (TODO: finish layout)
Parts:
- removed R9: 4,7k, rcl:R0805
- added C22: 100n, rcl:C0603
- R3: value 4.7k -> 43k
- R35: value 100k -> 33k
- R5: value 0 -> 1k
- R52: value 4.7k -> 1k
- R6: value 14k -> 8.2k
- moved R5 160.2 mm to (-22.7, -27.8), flipped to the top
Connections:
- removed net ADC_CAP_OV: IC4.5, R52.1, U5.7
- removed net FB_TRIG_LVL: C20.1, IC4.2, R3.1, R35.2
- removed net N$27: R6.2, R9.1
- new net TRIG_LVL_FB: C20.1, C22.2, IC4.2, R35.2, R5.1
- new net TRIG_LVL_OV: C22.1, IC4.6, R3.1, R5.2
- net +5V/3: no longer IC4.6
- net ADC_CAP: now also IC4.5
- net CAP_0V: now also R6.2; no longer R9.2
- net N$14: now also R4.2; no longer R5.2
- net N$15: now also R52.1, U5.7; no longer R4.2, R5.1
Routing:
- net ADC_CAP_OV: track 13.1 -> 0.00 mm
- net FB_TRIG_LVL: track 10.4 -> 0.00 mm
- net ADC_CAP: track 48.1 -> 56.4 mm
- net TRIG_LVL_FB: track 0.00 -> 3.84 mm
- net N$27: track 2.29 -> 0.00 mm
- net +5V/3: track 17.7 -> 15.6 mm
- net N$15: track 3.18 -> 4.63 mm
Changed lines of the file:
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@@
 </element>
 <element name="R4" library="rcl" package="R0805" value="240k" x="84.963" y="95.25" rot="MR0"/>
-<element name="R5" library="rcl" package="R0805" value="0" x="79.883" y="95.25" rot="MR0"/>
-<element name="R6" library="rcl" package="R0805" value="14k" x="81.788" y="75.946" rot="MR180"/>
-<element name="R9" library="rcl" package="R0805" value="4,7k" x="81.788" y="78.232" rot="MR0"/>
+<element name="R6" library="rcl" package="R0805" value="8.2k" x="81.788" y="75.946" rot="MR180"/>
 <element name="R10" library="rcl" package="R1206" value="1M, 1%" x="119.38" y="93.726" rot="MR270"/>
 <element name="D3" library="diode" package="TO236" value="SMD ZD 12" x="88.9" y="76.454"/>
@@
 <element name="C44" library="rcl" package="C0603" value="10p" x="88.265" y="74.93" rot="MR90"/>
 <element name="C46" library="rcl" package="C0603" value="10p" x="88.519" y="56.642" rot="MR270"/>
-<element name="R52" library="rcl" package="R0805" value="4.7k" x="86.106" y="56.642" rot="MR270"/>
+<element name="R52" library="rcl" package="R0805" value="1k" x="86.106" y="56.642" rot="MR270"/>
 <element name="D8" library="diode" package="TO236" value="BZX84-A5V1" x="83.058" y="56.642" rot="MR180"/>
 <element name="IC4" library="linear" package="SO08" value="MCP602-I/SN" x="91.567" y="49.276" rot="MR0"/>
@@
 <element name="R38" library="rcl" package="R1210" value="" x="120.65" y="44.704" rot="MR0"/>
 <element name="R39" library="rcl" package="R1210" value="" x="120.65" y="41.656" rot="MR0"/>
-<element name="R3" library="rcl" package="R0805" value="4.7k" x="87.503" y="49.276" rot="MR90"/>
-<element name="R35" library="rcl" package="R0805" value="100k" x="85.344" y="49.276" rot="MR270"/>
+<element name="R3" library="rcl" package="R0805" value="43k" x="87.503" y="49.276" rot="MR90"/>
+<element name="R35" library="rcl" package="R0805" value="33k" x="85.344" y="49.276" rot="MR270"/>
 <element name="C20" library="rcl" package="C0603" value="100n" x="83.312" y="49.276" rot="MR90"/>
+<element name="R5" library="rcl" package="R0805" value="1k" x="-22.733" y="-27.813"/>
+<element name="C22" library="rcl" package="C0603" value="100n" x="-21.971" y="-33.274"/>
 </elements>
 <signals>
@@
 <contactref element="RJ_1" pad="P$1"/>
 <contactref element="R35" pad="1"/>
-<contactref element="C20" pad="2"/>
 <contactref element="D8" pad="A"/>
 <contactref element="C57" pad="2"/>
+<contactref element="C20" pad="2"/>
 </signal>
 <signal name="SCK_3V">
@@
 <contactref element="C14" pad="2"/>
 <contactref element="C43" pad="2"/>
-<contactref element="R9" pad="2"/>
 <contactref element="H2" pad="B3,0"/>
 <contactref element="C44" pad="2"/>
@@
 <via x="82.677" y="91.186" extent="1-16" drill="0.5"/>
 <via x="75.311" y="97.663" extent="1-16" drill="0.5"/>
+<contactref element="R6" pad="2"/>
+<wire x1="82.638" y1="73.914" x2="82.738" y2="75.946" width="0" layer="19" extent="16-16"/>
 </signal>
 <signal name="CAP_12V">
@@
 <wire x1="81.915" y1="51.562" x2="81.915" y2="46.609" width="0.254" layer="16"/>
 <wire x1="81.915" y1="46.609" x2="83.693" y2="44.831" width="0.254" layer="16"/>
+<contactref element="IC4" pad="5"/>
+<wire x1="86.299" y1="57.592" x2="87.249" y2="56.642" width="0.254" layer="16"/>
+<wire x1="87.249" y1="56.642" x2="87.249" y2="54.991" width="0.254" layer="16"/>
+<wire x1="87.249" y1="54.991" x2="87.503" y2="54.737" width="0.254" layer="16"/>
+<wire x1="87.503" y1="54.737" x2="89.408" y2="54.737" width="0.254" layer="16"/>
+<wire x1="89.408" y1="54.737" x2="89.662" y2="54.483" width="0.254" layer="16"/>
+<wire x1="89.662" y1="54.483" x2="89.662" y2="51.876" width="0.254" layer="16"/>
+<wire x1="86.106" y1="55.692" x2="87.249" y2="54.991" width="0" layer="19" extent="16-16"/>
 </signal>
 <signal name="ÜBERSPANNUNG">
@@
 <contactref element="C39" pad="1"/>
 <contactref element="D14" pad="C"/>
-<contactref element="IC4" pad="6"/>
 <contactref element="C37" pad="1"/>
-<wire x1="90.932" y1="51.876" x2="90.932" y2="49.784" width="0.254" layer="16"/>
 <via x="90.932" y="49.784" extent="1-16" drill="0.5"/>
 <contactref element="R3" pad="2"/>
@@
 <signal name="N$14">
 <contactref element="R6" pad="1"/>
-<contactref element="R5" pad="2"/>
 <contactref element="U5" pad="12"/>
 <contactref element="C43" pad="1"/>
@@
 <wire x1="79.756" y1="75.946" x2="79.121" y2="76.581" width="0.4064" layer="16"/>
 <wire x1="79.121" y1="76.581" x2="79.121" y2="95.062" width="0.4064" layer="16"/>
-<wire x1="79.121" y1="95.062" x2="78.933" y2="95.25" width="0.4064" layer="16"/>
-</signal>
-<signal name="N$15">
-<contactref element="R5" pad="1"/>
 <contactref element="R4" pad="2"/>
-<wire x1="80.833" y1="95.25" x2="84.013" y2="95.25" width="0.4064" layer="16"/>
+<wire x1="79.121" y1="95.062" x2="84.013" y2="95.25" width="0" layer="19" extent="16-16"/>
 </signal>
 <signal name="N$21">
@@
 <contactref element="U5" pad="10"/>
 <wire x1="85.979" y1="70.6882" x2="84.709" y2="70.6882" width="0.4064" layer="16"/>
-</signal>
-<signal name="N$27">
-<contactref element="R6" pad="2"/>
-<contactref element="R9" pad="1"/>
-<wire x1="82.738" y1="78.232" x2="82.738" y2="75.946" width="0.4064" layer="16"/>
 </signal>
 <signal name="N$35">
@@
 <contactref element="C46" pad="1"/>
 <wire x1="88.519" y1="61.6458" x2="88.519" y2="57.492" width="0.4064" layer="16"/>
-</signal>
-<signal name="ADC_CAP_OV">
-<contactref element="U5" pad="7"/>
-<contactref element="R52" pad="1"/>
-<contactref element="IC4" pad="5"/>
-<wire x1="84.709" y1="61.6458" x2="84.709" y2="58.989" width="0.4064" layer="16"/>
-<wire x1="84.709" y1="58.989" x2="86.106" y2="57.592" width="0.4064" layer="16"/>
-<wire x1="86.106" y1="57.592" x2="86.299" y2="57.592" width="0.254" layer="16"/>
-<wire x1="86.299" y1="57.592" x2="87.249" y2="56.642" width="0.254" layer="16"/>
-<wire x1="87.249" y1="56.642" x2="87.249" y2="54.991" width="0.254" layer="16"/>
-<wire x1="87.249" y1="54.991" x2="87.503" y2="54.737" width="0.254" layer="16"/>
-<wire x1="87.503" y1="54.737" x2="89.408" y2="54.737" width="0.254" layer="16"/>
-<wire x1="89.408" y1="54.737" x2="89.662" y2="54.483" width="0.254" layer="16"/>
-<wire x1="89.662" y1="54.483" x2="89.662" y2="51.876" width="0.254" layer="16"/>
 </signal>
 <signal name="N$86">
@@
 <wire x1="119.25" y1="51.054" x2="119.25" y2="48.006" width="0.8128" layer="16"/>
 </signal>
-<signal name="FB_TRIG_LVL">
-<contactref element="R3" pad="1"/>
+<signal name="TRIG_LVL_FB">
 <contactref element="R35" pad="2"/>
 <contactref element="IC4" pad="2"/>
@@
 <wire x1="85.344" y1="48.326" x2="83.539" y2="48.326" width="0.254" layer="16"/>
 <wire x1="83.539" y1="48.326" x2="83.312" y2="48.426" width="0.254" layer="16"/>
-<wire x1="85.344" y1="48.326" x2="87.503" y2="48.326" width="0.254" layer="16"/>
-<wire x1="87.503" y1="48.326" x2="91.882" y2="48.326" width="0.254" layer="16"/>
 <wire x1="91.882" y1="48.326" x2="92.202" y2="48.006" width="0.254" layer="16"/>
 <wire x1="92.202" y1="48.006" x2="92.202" y2="46.676" width="0.254" layer="16"/>
+<contactref element="R5" pad="1"/>
+<contactref element="C22" pad="2"/>
+<wire x1="85.344" y1="48.326" x2="91.882" y2="48.326" width="0" layer="19" extent="16-16"/>
+<wire x1="-23.683" y1="-27.813" x2="83.312" y2="48.426" width="0" layer="19" extent="1-16"/>
+<wire x1="-21.121" y1="-33.274" x2="-23.683" y2="-27.813" width="0" layer="19" extent="1-1"/>
+</signal>
+<signal name="N$15">
+<contactref element="U5" pad="7"/>
+<contactref element="R52" pad="1"/>
+<wire x1="84.709" y1="61.6458" x2="84.709" y2="58.989" width="0.4064" layer="16"/>
+<wire x1="84.709" y1="58.989" x2="86.106" y2="57.592" width="0.4064" layer="16"/>
+</signal>
+<signal name="TRIG_LVL_OV">
+<contactref element="R3" pad="1"/>
+<contactref element="R5" pad="2"/>
+<contactref element="C22" pad="1"/>
+<contactref element="IC4" pad="6"/>
+<wire x1="87.503" y1="48.326" x2="90.932" y2="51.876" width="0" layer="19" extent="16-16"/>
+<wire x1="-21.783" y1="-27.813" x2="87.503" y2="48.326" width="0" layer="19" extent="1-16"/>
+<wire x1="-22.821" y1="-33.274" x2="-21.783" y2="-27.813" width="0" layer="19" extent="1-1"/>
 </signal>
 </signals>
