File: kicker/rekick2017/pcb/rekick2017-v0.2.sch (EAGLE design)
At the start: 184 parts, among them IC1 SN74LVC1G02DBVR, IC2 4043D, IC3 LM1117, IC4 MCP602-I/SN, P1 39-30-06_S, P2 39-30-08_S, Q1 16MHz, Q2 IKW40N120T2FKSA1, Q3 PSMN7R8-120PS, Q4 PSMN7R8-120PS, Q5 IPD90P04P4L, Q6 IRF840, T1 BC859, T5 IRLML6344TRPBF, U1 TXB0108PWR, U2 R-7805, U3 R-7812, U4 R-7805, U5 ADUM4190BRIZ

Commit message: corrected fb-loop
Parts:
- removed R21: 180k, rcl:R-EU_R0805
- removed R25: 56k, rcl:R-EU_R0805
- removed R26: 4.7k, rcl:R-EU_R0805
- added C20: 100n, rcl:C-EUC0603
- added R3: 4.7k, rcl:R-EU_R0805
- added R35: 100k, rcl:R-EU_R0805
Connections:
- removed net FB_OV: IC4A.+IN, R21.1, R25.2
- removed net N$34: R25.1, R26.2
- new net FB_TRIG_LVL: C20.1, IC4A.-IN, R3.1, R35.2
- net +5V/3: now also R3.2
- net ADC_CAP: now also IC4A.+IN; no longer R21.2
- net GND: now also C20.2, R35.1; no longer R26.1
- net N$3: no longer IC4A.-IN
Other:
- moved on the sheet: R52
Changed lines of the file:
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@@
 <part name="GND10" library="supply1" deviceset="GND" device=""/>
 <part name="SUPPLY6" library="supply2" deviceset="0V" device="" value="CAP_0V"/>
-<part name="R21" library="rcl" deviceset="R-EU_" device="R0805" value="180k"/>
-<part name="R25" library="rcl" deviceset="R-EU_" device="R0805" value="56k"/>
-<part name="R26" library="rcl" deviceset="R-EU_" device="R0805" value="4.7k"/>
 <part name="GND19" library="supply1" deviceset="GND" device=""/>
 <part name="R29" library="rcl" deviceset="R-EU_" device="R0805" value="5,6k"/>
@@
 <part name="R38" library="rcl" deviceset="R-EU_" device="R1210"/>
 <part name="R39" library="rcl" deviceset="R-EU_" device="R1210"/>
+<part name="R3" library="rcl" deviceset="R-EU_" device="R0805" value="4.7k"/>
+<part name="R35" library="rcl" deviceset="R-EU_" device="R0805" value="100k"/>
+<part name="GND14" library="supply1" deviceset="GND" device=""/>
+<part name="SUPPLY10" library="supply2" deviceset="+5V/3" device=""/>
+<part name="C20" library="rcl" deviceset="C-EU" device="C0603" value="100n"/>
 </parts>
 <sheets>
@@
 <instance part="C44" gate="G$1" x="109.22" y="106.68"/>
 <instance part="C46" gate="G$1" x="114.3" y="106.68"/>
-<instance part="R52" gate="G$1" x="116.84" y="132.08"/>
+<instance part="R52" gate="G$1" x="119.38" y="132.08"/>
 <instance part="D8" gate="G$1" x="129.54" y="121.92" rot="R90"/>
 <instance part="C57" gate="G$1" x="137.16" y="121.92"/>
 <instance part="GND10" gate="1" x="114.3" y="93.98"/>
 <instance part="SUPPLY6" gate="0V" x="109.22" y="91.44"/>
-<instance part="R21" gate="G$1" x="149.86" y="124.46" rot="R90"/>
-<instance part="R25" gate="G$1" x="149.86" y="109.22" rot="R90"/>
-<instance part="R26" gate="G$1" x="149.86" y="93.98" rot="R90"/>
-<instance part="GND19" gate="1" x="142.24" y="81.28"/>
+<instance part="GND19" gate="1" x="134.62" y="93.98"/>
 </instances>
 <busses>
@@
 </segment>
 <segment>
-<pinref part="D8" gate="G$1" pin="A"/>
-<wire x1="129.54" y1="99.06" x2="137.16" y2="99.06" width="0.1524" layer="91"/>
-<pinref part="C57" gate="G$1" pin="2"/>
-<pinref part="R26" gate="G$1" pin="1"/>
-<wire x1="149.86" y1="88.9" x2="149.86" y2="86.36" width="0.1524" layer="91"/>
-<wire x1="149.86" y1="86.36" x2="142.24" y2="86.36" width="0.1524" layer="91"/>
-<wire x1="142.24" y1="86.36" x2="137.16" y2="86.36" width="0.1524" layer="91"/>
-<wire x1="137.16" y1="86.36" x2="137.16" y2="99.06" width="0.1524" layer="91"/>
-<junction x="137.16" y="99.06"/>
-<pinref part="GND19" gate="1" pin="GND"/>
-<wire x1="142.24" y1="83.82" x2="142.24" y2="86.36" width="0.1524" layer="91"/>
-<junction x="142.24" y="86.36"/>
-<wire x1="129.54" y1="119.38" x2="129.54" y2="99.06" width="0.1524" layer="91"/>
-<wire x1="137.16" y1="116.84" x2="137.16" y2="99.06" width="0.1524" layer="91"/>
-</segment>
-<segment>
 <pinref part="GND20" gate="1" pin="GND"/>
 <wire x1="38.1" y1="127" x2="38.1" y2="129.54" width="0.1524" layer="91"/>
@@
 <wire x1="38.1" y1="129.54" x2="48.26" y2="129.54" width="0.1524" layer="91"/>
 <junction x="48.26" y="129.54"/>
+</segment>
+<segment>
+<pinref part="D8" gate="G$1" pin="A"/>
+<wire x1="129.54" y1="99.06" x2="134.62" y2="99.06" width="0.1524" layer="91"/>
+<pinref part="C57" gate="G$1" pin="2"/>
+<wire x1="134.62" y1="99.06" x2="137.16" y2="99.06" width="0.1524" layer="91"/>
+<wire x1="129.54" y1="119.38" x2="129.54" y2="99.06" width="0.1524" layer="91"/>
+<wire x1="137.16" y1="116.84" x2="137.16" y2="99.06" width="0.1524" layer="91"/>
+<wire x1="134.62" y1="99.06" x2="134.62" y2="96.52" width="0.1524" layer="91"/>
+<junction x="134.62" y="99.06"/>
+<pinref part="GND19" gate="1" pin="GND"/>
 </segment>
 </net>
@@
 <pinref part="R52" gate="G$1" pin="1"/>
 <wire x1="106.68" y1="132.08" x2="109.22" y2="132.08" width="0.1524" layer="91"/>
-<wire x1="109.22" y1="132.08" x2="111.76" y2="132.08" width="0.1524" layer="91"/>
-<wire x1="109.22" y1="132.08" x2="109.22" y2="147.32" width="0.1524" layer="91"/>
+<wire x1="109.22" y1="132.08" x2="114.3" y2="132.08" width="0.1524" layer="91"/>
+<wire x1="109.22" y1="132.08" x2="109.22" y2="139.7" width="0.1524" layer="91"/>
 <junction x="109.22" y="132.08"/>
-<wire x1="109.22" y1="147.32" x2="139.7" y2="147.32" width="0.1524" layer="91"/>
-<label x="139.7" y="147.32" size="1.778" layer="95" xref="yes"/>
+<wire x1="109.22" y1="139.7" x2="142.24" y2="139.7" width="0.1524" layer="91"/>
+<label x="142.24" y="139.7" size="1.778" layer="95" xref="yes"/>
 </segment>
 </net>
@@
 <segment>
 <pinref part="R52" gate="G$1" pin="2"/>
-<wire x1="154.94" y1="132.08" x2="149.86" y2="132.08" width="0.1524" layer="91"/>
-<label x="154.94" y="132.08" size="1.778" layer="95" xref="yes"/>
+<label x="142.24" y="132.08" size="1.778" layer="95" xref="yes"/>
 <pinref part="D8" gate="G$1" pin="C"/>
-<wire x1="149.86" y1="132.08" x2="137.16" y2="132.08" width="0.1524" layer="91"/>
+<wire x1="142.24" y1="132.08" x2="137.16" y2="132.08" width="0.1524" layer="91"/>
 <wire x1="129.54" y1="132.08" x2="137.16" y2="132.08" width="0.1524" layer="91"/>
-<wire x1="137.16" y1="132.08" x2="121.92" y2="132.08" width="0.1524" layer="91"/>
+<wire x1="137.16" y1="132.08" x2="124.46" y2="132.08" width="0.1524" layer="91"/>
 <wire x1="129.54" y1="124.46" x2="129.54" y2="132.08" width="0.1524" layer="91"/>
 <junction x="129.54" y="132.08"/>
@@
 <wire x1="137.16" y1="124.46" x2="137.16" y2="132.08" width="0.1524" layer="91"/>
 <junction x="137.16" y="132.08"/>
-<pinref part="R21" gate="G$1" pin="2"/>
-<wire x1="149.86" y1="129.54" x2="149.86" y2="132.08" width="0.1524" layer="91"/>
-<junction x="149.86" y="132.08"/>
-</segment>
-</net>
-<net name="FB_OV" class="0">
-<segment>
-<pinref part="R21" gate="G$1" pin="1"/>
-<pinref part="R25" gate="G$1" pin="2"/>
-<wire x1="149.86" y1="119.38" x2="149.86" y2="116.84" width="0.1524" layer="91"/>
-<wire x1="149.86" y1="116.84" x2="149.86" y2="114.3" width="0.1524" layer="91"/>
-<wire x1="149.86" y1="116.84" x2="154.94" y2="116.84" width="0.1524" layer="91"/>
-<junction x="149.86" y="116.84"/>
-<label x="154.94" y="116.84" size="1.778" layer="95" xref="yes"/>
-</segment>
-</net>
-<net name="N$34" class="0">
-<segment>
-<pinref part="R25" gate="G$1" pin="1"/>
-<pinref part="R26" gate="G$1" pin="2"/>
-<wire x1="149.86" y1="104.14" x2="149.86" y2="99.06" width="0.1524" layer="91"/>
 </segment>
 </net>
@@
 <instance part="R33" gate="G$1" x="66.04" y="121.92"/>
 <instance part="T4" gate="A" x="116.84" y="68.58"/>
+<instance part="R3" gate="G$1" x="43.18" y="160.02" rot="R90"/>
+<instance part="R35" gate="G$1" x="43.18" y="144.78" rot="R90"/>
+<instance part="GND14" gate="1" x="43.18" y="134.62"/>
+<instance part="SUPPLY10" gate="G$1" x="43.18" y="170.18"/>
+<instance part="C20" gate="G$1" x="50.8" y="144.78"/>
 </instances>
 <busses>
@@
 <wire x1="50.8" y1="22.86" x2="50.8" y2="25.4" width="0.1524" layer="91"/>
 </segment>
+<segment>
+<pinref part="R35" gate="G$1" pin="1"/>
+<pinref part="GND14" gate="1" pin="GND"/>
+<wire x1="43.18" y1="139.7" x2="43.18" y2="137.16" width="0.1524" layer="91"/>
+<pinref part="C20" gate="G$1" pin="2"/>
+<wire x1="43.18" y1="139.7" x2="50.8" y2="139.7" width="0.1524" layer="91"/>
+<junction x="43.18" y="139.7"/>
+</segment>
 </net>
 <net name="+5V" class="0">
@@
 <pinref part="IC4" gate="B" pin="-IN"/>
 <wire x1="40.64" y1="104.14" x2="35.56" y2="104.14" width="0.1524" layer="91"/>
+</segment>
+<segment>
+<pinref part="SUPPLY10" gate="G$1" pin="+5V/3"/>
+<pinref part="R3" gate="G$1" pin="2"/>
+<wire x1="43.18" y1="167.64" x2="43.18" y2="165.1" width="0.1524" layer="91"/>
 </segment>
 </net>
@@
 <segment>
 <pinref part="IC4" gate="A" pin="OUT"/>
-<wire x1="55.88" y1="121.92" x2="58.42" y2="121.92" width="0.1524" layer="91"/>
-<wire x1="58.42" y1="121.92" x2="58.42" y2="114.3" width="0.1524" layer="91"/>
-<wire x1="58.42" y1="114.3" x2="38.1" y2="114.3" width="0.1524" layer="91"/>
-<wire x1="38.1" y1="114.3" x2="38.1" y2="119.38" width="0.1524" layer="91"/>
-<pinref part="IC4" gate="A" pin="-IN"/>
-<wire x1="38.1" y1="119.38" x2="40.64" y2="119.38" width="0.1524" layer="91"/>
-<wire x1="58.42" y1="121.92" x2="60.96" y2="121.92" width="0.1524" layer="91"/>
-<junction x="58.42" y="121.92"/>
+<wire x1="55.88" y1="121.92" x2="60.96" y2="121.92" width="0.1524" layer="91"/>
 <pinref part="R33" gate="G$1" pin="1"/>
 </segment>
 </net>
-<net name="FB_OV" class="0">
+<net name="FB" class="0">
+<segment>
+<pinref part="R33" gate="G$1" pin="2"/>
+<wire x1="71.12" y1="121.92" x2="73.66" y2="121.92" width="0.1524" layer="91"/>
+<label x="73.66" y="121.92" size="1.778" layer="95" xref="yes"/>
+</segment>
+</net>
+<net name="ADC_CAP" class="0">
 <segment>
 <pinref part="IC4" gate="A" pin="+IN"/>
@@
 </segment>
 </net>
-<net name="FB" class="0">
-<segment>
-<pinref part="R33" gate="G$1" pin="2"/>
-<wire x1="71.12" y1="121.92" x2="73.66" y2="121.92" width="0.1524" layer="91"/>
-<label x="73.66" y="121.92" size="1.778" layer="95" xref="yes"/>
-</segment>
-</net>
+<net name="FB_TRIG_LVL" class="0">
+<segment>
+<pinref part="R3" gate="G$1" pin="1"/>
+<pinref part="R35" gate="G$1" pin="2"/>
+<wire x1="43.18" y1="154.94" x2="43.18" y2="152.4" width="0.1524" layer="91"/>
+<wire x1="43.18" y1="152.4" x2="43.18" y2="149.86" width="0.1524" layer="91"/>
+<junction x="43.18" y="152.4"/>
+<wire x1="43.18" y1="152.4" x2="50.8" y2="152.4" width="0.1524" layer="91"/>
+<label x="55.88" y="152.4" size="1.778" layer="95" xref="yes"/>
+<pinref part="C20" gate="G$1" pin="1"/>
+<wire x1="50.8" y1="152.4" x2="55.88" y2="152.4" width="0.1524" layer="91"/>
+<wire x1="50.8" y1="147.32" x2="50.8" y2="152.4" width="0.1524" layer="91"/>
+<junction x="50.8" y="152.4"/>
+</segment>
+<segment>
+<pinref part="IC4" gate="A" pin="-IN"/>
+<wire x1="35.56" y1="119.38" x2="40.64" y2="119.38" width="0.1524" layer="91"/>
+<label x="35.56" y="119.38" size="1.778" layer="95" rot="R180" xref="yes"/>
+</segment>
+</net>

Commit message: kicker 2017 v0.2 final
Connections:
- net CAP_+12V renamed CAP_12V
Changed lines of the file:
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@@
 <part name="GND8" library="supply1" deviceset="GND" device=""/>
 <part name="SUPPLY2" library="supply2" deviceset="0V" device="" value="CAP_0V"/>
-<part name="SUPPLY5" library="supply2" deviceset="+12V" device="" value="CAP_+12V"/>
 <part name="SUPPLY9" library="supply2" deviceset="0V" device="" value="CAP_0V"/>
 <part name="D9" library="diode" deviceset="BYT08P" device="" value="STTH810D"/>
@@
 <part name="R14" library="rcl" deviceset="R-EU_" device="R0805" value="390"/>
 <part name="FRAME7" library="frames" deviceset="A4L-LOC" device=""/>
-<part name="SUPPLY12" library="supply2" deviceset="+12V" device="" value="CAP_+12V"/>
 <part name="SUPPLY15" library="supply2" deviceset="0V" device="" value="CAP_0V"/>
 <part name="GND25" library="supply1" deviceset="GND" device=""/>
@@
 <part name="U$5" library="Si8261" deviceset="SI8261ABC" device=""/>
 <part name="U$6" library="Si8261" deviceset="SI8261ABC" device=""/>
-<part name="SUPPLY16" library="supply2" deviceset="+12V" device="" value="CAP_+12V"/>
 <part name="SUPPLY17" library="supply2" deviceset="0V" device="" value="CAP_0V"/>
 <part name="R15" library="rcl" deviceset="R-EU_" device="R0805" value="5.6k"/>
@@
 <part name="SUPPLY11" library="supply2" deviceset="0V" device="" value="CAP_0V"/>
 <part name="GND20" library="supply1" deviceset="GND" device=""/>
-<part name="SUPPLY14" library="supply2" deviceset="+12V" device="" value="CAP_+12V"/>
 <part name="P+20" library="supply1" deviceset="+12V" device=""/>
 <part name="C43" library="rcl" deviceset="C-EU" device="C0603" value="100n"/>
@@
 <instance part="GND8" gate="1" x="175.26" y="33.02"/>
 <instance part="SUPPLY2" gate="0V" x="238.76" y="35.56"/>
-<instance part="SUPPLY5" gate="+12V" x="218.44" y="53.34"/>
 <instance part="LED9" gate="G$1" x="238.76" y="48.26"/>
 <instance part="R49" gate="G$1" x="228.6" y="50.8" rot="R180"/>
@@
 </segment>
 </net>
-<net name="CAP_+12V" class="0">
+<net name="CAP_12V" class="0">
 <segment>
 <pinref part="U$4" gate="G$1" pin="+U_OUT"/>
-<pinref part="SUPPLY5" gate="+12V" pin="+12V"/>
 <wire x1="210.82" y1="50.8" x2="218.44" y2="50.8" width="0.1524" layer="91"/>
 <junction x="218.44" y="50.8"/>
@@
 <pinref part="C19" gate="G$1" pin="1"/>
 <wire x1="218.44" y1="48.26" x2="218.44" y2="50.8" width="0.1524" layer="91"/>
+<wire x1="218.44" y1="50.8" x2="218.44" y2="53.34" width="0.1524" layer="91"/>
+<label x="218.44" y="53.34" size="1.778" layer="95" rot="R90" xref="yes"/>
 </segment>
 </net>
@@
 <instance part="R17" gate="G$1" x="48.26" y="152.4" rot="R90"/>
 <instance part="U$6" gate="G$1" x="76.2" y="142.24"/>
-<instance part="SUPPLY16" gate="+12V" x="96.52" y="152.4"/>
 <instance part="SUPPLY17" gate="0V" x="96.52" y="127"/>
 <instance part="R18" gate="G$1" x="119.38" y="139.7"/>
@@
 </segment>
 </net>
-<net name="CAP_+12V" class="0">
-<segment>
-<pinref part="SUPPLY16" gate="+12V" pin="+12V"/>
+<net name="CAP_12V" class="0">
+<segment>
 <wire x1="96.52" y1="147.32" x2="96.52" y2="149.86" width="0.1524" layer="91"/>
 <wire x1="93.98" y1="147.32" x2="96.52" y2="147.32" width="0.1524" layer="91"/>
@@
 <pinref part="C31" gate="G$1" pin="1"/>
 <wire x1="101.6" y1="142.24" x2="101.6" y2="147.32" width="0.1524" layer="91"/>
+<label x="96.52" y="149.86" size="1.778" layer="95" rot="R90" xref="yes"/>
 </segment>
 </net>
@@
 <instance part="SUPPLY11" gate="0V" x="43.18" y="124.46"/>
 <instance part="GND20" gate="1" x="38.1" y="124.46"/>
-<instance part="SUPPLY14" gate="+12V" x="68.58" y="137.16"/>
 <instance part="P+20" gate="1" x="63.5" y="139.7"/>
 <instance part="C43" gate="G$1" x="20.32" y="109.22"/>
@@
 </segment>
 </net>
-<net name="CAP_+12V" class="0">
-<segment>
-<pinref part="SUPPLY14" gate="+12V" pin="+12V"/>
+<net name="CAP_12V" class="0">
+<segment>
 <pinref part="C14" gate="G$1" pin="1"/>
 <wire x1="66.04" y1="129.54" x2="68.58" y2="129.54" width="0.1524" layer="91"/>
@@
 <junction x="68.58" y="129.54"/>
 <pinref part="U5" gate="A" pin="VDD2"/>
+<label x="68.58" y="134.62" size="1.778" layer="95" rot="R90" xref="yes"/>
 </segment>
 </net>
@@
 <instance part="SUPPLY18" gate="G$1" x="33.02" y="104.14" rot="R90"/>
 <instance part="R14" gate="G$1" x="35.56" y="68.58"/>
-<instance part="SUPPLY12" gate="+12V" x="86.36" y="78.74"/>
 <instance part="SUPPLY15" gate="0V" x="86.36" y="53.34"/>
 <instance part="U$5" gate="G$1" x="66.04" y="68.58"/>
@@
 </segment>
 </net>
-<net name="CAP_+12V" class="0">
-<segment>
-<pinref part="SUPPLY12" gate="+12V" pin="+12V"/>
+<net name="CAP_12V" class="0">
+<segment>
 <wire x1="86.36" y1="73.66" x2="86.36" y2="76.2" width="0.1524" layer="91"/>
 <pinref part="U$5" gate="G$1" pin="VDD"/>
@@
 <pinref part="C30" gate="G$1" pin="1"/>
 <wire x1="91.44" y1="68.58" x2="91.44" y2="73.66" width="0.1524" layer="91"/>
-</segment>
-</net>
+<label x="86.36" y="76.2" size="1.778" layer="95" rot="R90" xref="yes"/>
+</segment>
+</net>

Commit message: rekick2017 0.2 (TODO: finish layout)
Parts:
- removed R9: 4,7k, rcl:R-EU_R0805
- added C22: 100n, rcl:C-EUC0603
- R3: value 4.7k -> 43k
- R35: value 100k -> 33k
- R5: value 0 -> 1k
- R52: value 4.7k -> 1k
- R6: value 14k -> 8.2k
Connections:
- removed net ADC_CAP_OV: IC4B.+IN, R52.1, U5.EAOUT1
- removed net FB_TRIG_LVL: C20.1, IC4A.-IN, R3.1, R35.2
- removed net N$27: R6.2, R9.1
- new net TRIG_LVL_FB: C20.1, C22.2, IC4A.-IN, R35.2, R5.1
- new net TRIG_LVL_OV: C22.1, IC4B.-IN, R3.1, R5.2
- net +5V/3: no longer IC4B.-IN
- net ADC_CAP: now also IC4B.+IN
- net CAP_0V: now also R6.2; no longer R9.2
- net N$14: now also R4.2; no longer R5.2
- net N$15: now also R52.1, U5.EAOUT1; no longer R4.2, R5.1
Other:
- moved on the sheet: C20, C43, C44, C46, C57, D8, IC4A, IC4B, R101, R33, R35, R4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
